File: pcb/stlink.kicad_pcb (KiCad board)
At the start: 4 copper layers, 35.5 x 20 mm, 40 parts, among them J1 USB_A, Q1 S9013, U1 XC6206P332MR, U2 STM32F103CBT6, Y1 8MHz

Commit message: Hmmm
Parts:
- U2: value STM32F103CBT6 -> GD32F103CBT6
- moved R8 12.9 mm to (119.2, 83.5), turned to 270 degrees
- moved R7 12.3 mm to (120.5, 83.5), turned to 270 degrees
- moved TP2 6.25 mm to (129.0, 83.5)
- moved R9 4.51 mm to (127.8, 94.8), turned to 270 degrees
- moved TP1 4.31 mm to (131.1, 83.5)
- moved TP4 4.22 mm to (125.0, 83.5)
- moved TP5 4.19 mm to (122.9, 83.5)
- moved TP3 2.25 mm to (127.0, 83.5)
- moved R11 1.59 mm to (121.5, 96.2), turned to 90 degrees
- moved R13 0.95 mm to (113.3, 96.8)
- moved R3 0.95 mm to (129.2, 90.2), turned to 180 degrees
- moved R10 0.90 mm to (120.2, 96.2), turned to 270 degrees
- moved C8 0.71 mm to (126.8, 94.8)
- moved R5 0.56 mm to (133.0, 94.5)
- moved Q1 0.50 mm to (130.8, 92.8)
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Connections:
- J1 pad 5: Net-(J1-Pad5) -> GND
Routing:
- net +5V: track 0.00 -> 29.8 mm, vias 0 -> 2
- net +3V3: track 0.00 -> 26.6 mm, vias 0 -> 9
- net T_DIO: track 0.00 -> 22.2 mm, vias 0 -> 2
- net T_CLK: track 0.00 -> 17.4 mm, vias 0 -> 1
- net T_SWO: track 0.00 -> 17.2 mm, vias 0 -> 1
- net LED: track 0.00 -> 16.8 mm, vias 0 -> 2
- net T_RST: track 0.00 -> 14.8 mm, vias 0 -> 2
- net RENUM: track 0.00 -> 13.7 mm, vias 0 -> 2
- net T_RX: track 0.00 -> 11.0 mm, vias 0 -> 2
- net D+: track 0.00 -> 9.67 mm, vias 0 -> 1
- net T_TX: track 0.00 -> 8.66 mm, vias 0 -> 1
- net DIO: track 0.00 -> 8.21 mm, vias 0 -> 1
- net D-: track 0.00 -> 8.20 mm, vias 0 -> 1
- net Net-(R10-Pad1): track 0.00 -> 8.17 mm, vias 0 -> 2
- net Net-(C2-Pad1): track 0.00 -> 7.42 mm
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Other:
- board text added: "+3V3"
- board text added: "+5V/+3.3V"
- board text added: "B0"
- board text added: "CLK"
- board text added: "CLK/DIO"
- board text added: "DIO"
- board text added: "GND"
- board text added: "JLCJLCJLCJLC"
- board text added: "PWR/GND"
- board text added: "STM32 Programmer rev. a"
- board text added: "SWO/RST"
- board text added: "TX/RX"

Commit message: Hmmm
Parts:
- moved C8 2.50 mm to (124.8, 96.2), turned to 90 degrees
- moved R9 2.30 mm to (126.0, 96.2)
- moved D1 0.50 mm to (130.8, 84.0)
Routing:
- net +3V3: track 26.6 -> 31.4 mm, vias 9 -> 11
- net T_DIO: track 22.2 -> 24.3 mm
- net GND: track 0.52 -> 2.33 mm, vias 12 -> 16
- net Net-(R9-Pad1): track 1.73 -> 3.47 mm
- net +5V: track 29.8 -> 30.3 mm

Commit message: Order rev a
Parts:
- added JP1: ~, Jumper:SolderJumper-3_P1.3mm_Bridged12_Pad1.0x1.5mm, B.Cu at (122.5, 94.8)
- R8: value NP -> DNP
- moved R9 2.75 mm to (128.8, 96.2), turned to 90 degrees
- moved C8 2.00 mm to (126.8, 96.2), turned to 270 degrees
- moved R10 1.75 mm to (122.0, 96.2)
- moved R2 1.75 mm to (123.5, 83.5)
- moved R11 1.00 mm to (120.5, 96.2)
- moved R7 0.75 mm to (121.2, 83.5)
Connections:
- R10 pad 2: +3V3 -> Net-(JP1-Pad2)
Routing:
- net T_PWR: track 0.00 -> 22.5 mm
- net Net-(JP1-Pad2): track 0.00 -> 2.79 mm, vias 0 -> 1
- net Net-(R10-Pad1): track 8.17 -> 10.4 mm
- net GND: track 2.33 -> 0.64 mm
- net T_DIO: track 24.3 -> 22.6 mm
- net Net-(R9-Pad1): track 3.47 -> 4.67 mm
- net Net-(R7-Pad2): track 6.50 -> 7.25 mm
