File: pcb/stlink.kicad_pcb (KiCad board)
At the start: 4 copper layers, 35.5 x 20 mm, 41 parts, among them J1 USB_A, Q1 S9013, U1 XC6206P332MR, U2 GD32F103CBT6, Y1 8MHz

Commit message: Hmmmm
Parts:
- D2: value GREEN -> BLUE
Other:
- board text added: "STM32 Programmer rev. b"
- board text removed: "STM32 Programmer rev. a"
Changed lines of the file:
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@@
   (title_block
     (title "STM32 Programmer")
-    (rev a)
+    (rev b)
     (company "Lars Boegild Thomsen")
     (comment 1 lbthomsen@gmail.com)
@@
       (effects (font (size 0.8 0.8) (thickness 0.15)))
     )
-    (fp_text value GREEN (at 0 1.43) (layer F.Fab)
+    (fp_text value BLUE (at 0 1.43) (layer F.Fab)
       (effects (font (size 1 1) (thickness 0.15)))
     )
@@
     (effects (font (size 0.8 0.8) (thickness 0.15)) (justify left mirror))
   )
-  (gr_text "STM32\nProgrammer\nrev. a" (at 132.588 90.932) (layer B.SilkS)
+  (gr_text "STM32\nProgrammer\nrev. b" (at 132.588 90.932) (layer B.SilkS)
     (effects (font (size 1 1) (thickness 0.15)) (justify left mirror))
   )

Commit message: Hmmmm
Routing:
- net T_PWR: track 22.5 -> 23.2 mm

Commit message: Hmmmm
Parts:
- moved J2 1.00 mm to (109.2, 90.0)
Routing:
- net T_RX: track 11.0 -> 12.3 mm
- net +5V: track 30.3 -> 31.4 mm
- net T_SWO: track 17.2 -> 18.2 mm
- net T_TX: track 8.66 -> 9.69 mm
- net T_PWR: track 23.2 -> 24.2 mm
- net T_DIO: track 22.6 -> 23.7 mm
- net T_CLK: track 17.4 -> 18.4 mm
- net T_RST: track 14.8 -> 15.7 mm
Other:
- board size 35.5 x 20 mm -> 36.5 x 20 mm

Commit message: Hmmm
Routing:
- net T_PWR: track 24.2 -> 23.5 mm
Changed lines of the file:
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@@
     (thickness 1.6)
     (drawings 46)
-    (tracks 290)
+    (tracks 288)
     (zones 0)
     (modules 41)
@@
   )
   (setup
-    (last_trace_width 0.2286)
+    (last_trace_width 0.1524)
     (user_trace_width 0.1524)
     (user_trace_width 0.2286)
@@
   (segment (start 121.478723 91.421277) (end 118.901063 91.421277) (width 0.2286) (layer B.Cu) (net 16))
   (segment (start 122.1 90.8) (end 121.478723 91.421277) (width 0.2286) (layer B.Cu) (net 16))
-  (segment (start 124.2714 93.25) (end 123.75 93.7714) (width 0.2286) (layer B.Cu) (net 17))
-  (segment (start 126.75 92.75) (end 126.25 93.25) (width 0.2286) (layer B.Cu) (net 17))
-  (segment (start 123.366701 88.366701) (end 126.75 91.75) (width 0.2286) (layer B.Cu) (net 17))
-  (segment (start 118.866701 88.366701) (end 123.366701 88.366701) (width 0.2286) (layer B.Cu) (net 17))
-  (segment (start 117 86.5) (end 118.866701 88.366701) (width 0.2286) (layer B.Cu) (net 17))
-  (segment (start 126.75 91.75) (end 126.75 92.75) (width 0.2286) (layer B.Cu) (net 17))
-  (segment (start 115.25 86.5) (end 117 86.5) (width 0.2286) (layer B.Cu) (net 17))
-  (segment (start 123.75 93.7714) (end 123.75 94.75) (width 0.2286) (layer B.Cu) (net 17))
-  (segment (start 126.25 93.25) (end 124.2714 93.25) (width 0.2286) (layer B.Cu) (net 17))
-  (segment (start 114.37 87.38) (end 115.25 86.5) (width 0.2286) (layer B.Cu) (net 17))
+  (segment (start 123.366701 88.366701) (end 113.706701 88.366701) (width 0.2286) (layer B.Cu) (net 17))
+  (segment (start 126.75 91.75) (end 123.366701 88.366701) (width 0.2286) (layer B.Cu) (net 17))
+  (segment (start 126.75 92.75) (end 126.75 91.75) (width 0.2286) (layer B.Cu) (net 17))
+  (segment (start 126.25 93.25) (end 126.75 92.75) (width 0.2286) (layer B.Cu) (net 17))
+  (segment (start 112.72 87.38) (end 110.58 87.38) (width 0.2286) (layer B.Cu) (net 17))
+  (segment (start 124.2714 93.25) (end 126.25 93.25) (width 0.2286) (layer B.Cu) (net 17))
   (segment (start 110.58 87.38) (end 110.5 87.46) (width 0.2286) (layer B.Cu) (net 17))
-  (segment (start 114.37 87.38) (end 110.58 87.38) (width 0.2286) (layer B.Cu) (net 17))
+  (segment (start 123.75 93.7714) (end 124.2714 93.25) (width 0.2286) (layer B.Cu) (net 17))
+  (segment (start 113.706701 88.366701) (end 112.72 87.38) (width 0.2286) (layer B.Cu) (net 17))
+  (segment (start 123.75 94.75) (end 123.75 93.7714) (width 0.2286) (layer B.Cu) (net 17))
   (via (at 125.4 88) (size 0.7) (drill 0.35) (layers F.Cu B.Cu) (net 18) (status 40000))
   (segment (start 126 88) (end 129 85) (width 0.2286) (layer B.Cu) (net 18))

Commit message: Cosmetic changes
Other:
- board text added: "3V3"
- board text added: "5V/3V3"
- board text added: "ST-Link Clone rev. b"
- board text removed: "+3V3"
- board text removed: "+5V/+3.3V"
- board text removed: "STM32 Programmer rev. b"
Changed lines of the file:
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@@
-(kicad_pcb (version 20171130) (host pcbnew 5.1.9+dfsg1-1)
+(kicad_pcb (version 20171130) (host pcbnew 5.99.0+really5.1.10+dfsg1-1+b1)
   (general
     (thickness 1.6)
@@
     (rev b)
     (company "Lars Boegild Thomsen")
-    (comment 1 lbthomsen@gmail.com)
+    (comment 1 lth@stm32world.com)
   )
   (layers
@@
     (effects (font (size 0.8 0.8) (thickness 0.15)) (justify left mirror))
   )
-  (gr_text +3V3 (at 131.064 84.328 90) (layer B.SilkS)
+  (gr_text 3V3 (at 131.064 84.328 90) (layer B.SilkS)
     (effects (font (size 0.8 0.8) (thickness 0.15)) (justify left mirror))
   )
-  (gr_text TX/RX (at 113.284 94.996) (layer B.SilkS)
+  (gr_text TX/RX (at 112.395 94.996) (layer B.SilkS)
     (effects (font (size 0.8 0.8) (thickness 0.15)) (justify right mirror))
   )
-  (gr_text SWO/RST (at 113.284 92.456) (layer B.SilkS)
+  (gr_text SWO/RST (at 112.395 92.456) (layer B.SilkS)
     (effects (font (size 0.8 0.8) (thickness 0.15)) (justify right mirror))
   )
-  (gr_text CLK/DIO (at 113.284 89.916) (layer B.SilkS)
+  (gr_text CLK/DIO (at 112.395 89.916) (layer B.SilkS)
     (effects (font (size 0.8 0.8) (thickness 0.15)) (justify right mirror))
   )
-  (gr_text PWR/GND (at 113.284 87.376) (layer B.SilkS)
+  (gr_text PWR/GND (at 112.395 87.376) (layer B.SilkS)
     (effects (font (size 0.8 0.8) (thickness 0.15)) (justify right mirror))
   )
-  (gr_text +5V/+3.3V (at 113.284 84.836) (layer B.SilkS)
+  (gr_text 5V/3V3 (at 112.395 84.836) (layer B.SilkS)
     (effects (font (size 0.8 0.8) (thickness 0.15)) (justify right mirror))
   )
@@
     (effects (font (size 0.8 0.8) (thickness 0.15)) (justify left mirror))
   )
-  (gr_text "STM32\nProgrammer\nrev. b" (at 132.588 90.932) (layer B.SilkS)
+  (gr_text "ST-Link Clone\nrev. b" (at 132.08 89.535) (layer B.SilkS)
     (effects (font (size 1 1) (thickness 0.15)) (justify left mirror))
   )

Commit message: Hmmmm
Parts:
- R5: value 33k -> 39k
Connections:
- U2 pad 11: Net-(U2-Pad11) -> unconnected-(U2-Pad11)
- U2 pad 14: Net-(U2-Pad14) -> unconnected-(U2-Pad14)
- U2 pad 15: Net-(U2-Pad15) -> unconnected-(U2-Pad15)
- U2 pad 16: Net-(U2-Pad16) -> unconnected-(U2-Pad16)
- U2 pad 17: Net-(U2-Pad17) -> unconnected-(U2-Pad17)
- U2 pad 19: Net-(U2-Pad19) -> unconnected-(U2-Pad19)
- U2 pad 20: Net-(U2-Pad20) -> unconnected-(U2-Pad20)
- U2 pad 21: Net-(U2-Pad21) -> unconnected-(U2-Pad21)
- U2 pad 22: Net-(U2-Pad22) -> unconnected-(U2-Pad22)
- U2 pad 28: Net-(U2-Pad28) -> unconnected-(U2-Pad28)
- U2 pad 29: Net-(U2-Pad29) -> unconnected-(U2-Pad29)
- U2 pad 39: Net-(U2-Pad39) -> unconnected-(U2-Pad39)
- U2 pad 4: Net-(U2-Pad4) -> unconnected-(U2-Pad4)
- U2 pad 40: Net-(U2-Pad40) -> unconnected-(U2-Pad40)
- U2 pad 41: Net-(U2-Pad41) -> unconnected-(U2-Pad41)
- U2 pad 42: Net-(U2-Pad42) -> unconnected-(U2-Pad42)
- U2 pad 43: Net-(U2-Pad43) -> unconnected-(U2-Pad43)
- U2 pad 45: Net-(U2-Pad45) -> unconnected-(U2-Pad45)
- U2 pad 46: Net-(U2-Pad46) -> unconnected-(U2-Pad46)
Other:
- net class Default removed

Commit message: Hmmmm
Parts:
- moved D1 0.18 mm to (130.8, 83.8)
- moved U1 0.15 mm to (132.1, 86.9)
- moved C5 0.13 mm to (129.2, 86.9)
Connections:
- C5 pad 1: +3V3 -> +5V
- C7 pad 1: +3V3 -> +5V
- TP1 pad 1: +3V3 -> +5V
- U1 pad 2: +3V3 -> +5V
- U2 pad 36: +3V3 -> +5V
Routing:
- net +5V: track 31.4 -> 45.6 mm, vias 2 -> 4
- net +3V3: track 31.4 -> 18.7 mm, vias 11 -> 8
- net GND: vias 16 -> 17
Other:
- board text added: "${TITLE} rev. ${REVISION}"
- board text removed: "ST-Link Clone rev. b"

Commit message: Hmmmm
Parts:
- U2: value GD32F103CBT6 -> STM32F103C8
Connections:
- C5 pad 1: +5V -> +3V3
- C7 pad 1: +5V -> +3V3
- TP1 pad 1: +5V -> +3V3
- U1 pad 2: +5V -> +3V3
- U2 pad 36: +5V -> +3V3
Routing:
- net +5V: track 45.6 -> 32.1 mm, vias 4 -> 2
- net +3V3: track 18.7 -> 30.8 mm, vias 8 -> 10
