File: pcb/stlink.sch (KiCad schematic (older format))
At the start: 40 parts, among them J1 USB_A, Q1 S9013, U1 XC6206P332MR, U2 STM32F103CBT6, Y1 8MHz

Commit message: Hmmm
Parts:
- U2: value STM32F103CBT6 -> GD32F103CBT6; LCSC C8304 -> C77979
Connections:
- net GND: now also J1.5 (Shield)
Other:
- moved on the sheet: C4, C5, C6, C7, C8, C9, U1

Commit message: Hmmm
Other:
- note added: "Decoupling"
- note added: "MCU"
- note added: "Power Supply"
- note added: "Programming Pins"
- note added: "Target Header"
- note added: "Two-color LED"
- note added: "USB Connector"
- moved on the sheet: C1, C2, C3, C4, C5, C6, C7, C8, C9, D1, D2, D3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

Commit message: Order rev a
Parts:
- added JP1: ~, Jumper:SolderJumper-3_P1.3mm_Bridged12_Pad1.0x1.5mm, symbol Jumper:SolderJumper_3_Bridged12
- R8: value NP -> DNP
Connections:
- net +3V3: now also JP1.1 (A); no longer R10.2
- net T_PWR: now also JP1.3 (B)
- new net: JP1.2 (C), R10.2
Other:
- moved on the sheet: C1, C2, C3, R1, R10, R11, R2, R7, R8, Y1

Commit message: Hmmm
Parts:
- added R14, R15, R16, R17, R18, R19: 22R, Resistor_SMD:R_0402_1005Metric, symbol Device:R
Connections:
- net T_CLK: now also R14.2; no longer J2.5 (Pin_5)
- net T_DIO: now also R17.1; no longer J2.6 (Pin_6)
- net T_RST: no longer J2.8 (Pin_8)
- net T_RX: now also R19.1; no longer J2.10 (Pin_10)
- net T_SWO: now also R15.2; no longer J2.7 (Pin_7)
- net T_TX: now also R16.2; no longer J2.9 (Pin_9)
- new net: J2.10 (Pin_10), R19.2
- new net: J2.5 (Pin_5), R14.1
- new net: J2.6 (Pin_6), R17.2
- new net: J2.7 (Pin_7), R15.1
- new net: J2.8 (Pin_8), R18.2
- new net: J2.9 (Pin_9), R16.1
Other:
- moved on the sheet: D2, D3, J2, R12, R13
