File: pcb/stlink.sch (KiCad schematic (older format))
At the start: 41 parts, among them J1 USB_A, Q1 S9013, U1 XC6206P332MR, U2 GD32F103CBT6, Y1 8MHz

Commit message: Hmmmm
Parts:
- D2: value GREEN -> BLUE; LCSC C72043 -> C72041
Other:
- note added: "USB Connection and renumeration circuitry"
- note removed: "USB Connector"
Changed lines of the file:
@@
 Title "STM32 Programmer"
 Date ""
-Rev "a"
+Rev "b"
 Comp "Lars Boegild Thomsen"
 Comment1 "lbthomsen@gmail.com"
@@
 P 7550 4750
 F 0 "D2" V 7589 4632 50  0000 R CNN
-F 1 "GREEN" V 7498 4632 50  0000 R CNN
+F 1 "BLUE" V 7498 4632 50  0000 R CNN
 F 2 "LED_SMD:LED_0603_1608Metric" H 7550 4750 50  0001 C CNN
 F 3 "~" H 7550 4750 50  0001 C CNN
-F 4 "C72043" V 7550 4750 50  0001 C CNN "LCSC"
+F 4 "C72041" V 7550 4750 50  0001 C CNN "LCSC"
 	1    7550 4750
 	0    -1   -1   0
@@
 	4200 650  4200 3100
 Text Notes 800  600  0    50   ~ 0
-USB Connector
+USB Connection and renumeration circuitry
 Text Notes 4450 600  0    50   ~ 0
 Power Supply

Commit message: Hmmmm
Other:
- moved on the sheet: C4, C5, Q1, R3, R4, R5, R6

Commit message: Hmmm
Other:
- note added: "Works with STM32F103C8,\nSTM32F103CB\nor GD32F103CB"
- moved on the sheet: C4, C5
Changed lines of the file:
@@
 U 1 1 5EF85B23
 P 5400 1650
-F 0 "U1" H 5400 1892 50  0000 C CNN
-F 1 "XC6206P332MR" H 5400 1801 50  0000 C CNN
+F 0 "U1" H 5250 1800 50  0000 C CNN
+F 1 "XC6206P332MR" H 5650 1800 50  0000 C CNN
 F 2 "Package_TO_SOT_SMD:SOT-23" H 5400 1875 50  0001 C CIN
 F 3 "https://datasheet.lcsc.com/szlcsc/Torex-Semicon-XC6206P332MR_C5446.pdf" H 5400 1650 50  0001 C CNN
@@
 L power:+3V3 #PWR018
 U 1 1 5EF86316
-P 5950 1550
-F 0 "#PWR018" H 5950 1400 50  0001 C CNN
-F 1 "+3V3" H 5965 1723 50  0000 C CNN
-F 2 "" H 5950 1550 50  0001 C CNN
-F 3 "" H 5950 1550 50  0001 C CNN
-	1    5950 1550
+P 6100 1550
+F 0 "#PWR018" H 6100 1400 50  0001 C CNN
+F 1 "+3V3" H 6115 1723 50  0000 C CNN
+F 2 "" H 6100 1550 50  0001 C CNN
+F 3 "" H 6100 1550 50  0001 C CNN
+	1    6100 1550
 	1    0    0    -1
 $EndComp
@@
 L power:+5V #PWR014
 U 1 1 5EF86831
-P 4850 1550
-F 0 "#PWR014" H 4850 1400 50  0001 C CNN
-F 1 "+5V" H 4865 1723 50  0000 C CNN
-F 2 "" H 4850 1550 50  0001 C CNN
-F 3 "" H 4850 1550 50  0001 C CNN
-	1    4850 1550
+P 4650 1550
+F 0 "#PWR014" H 4650 1400 50  0001 C CNN
+F 1 "+5V" H 4665 1723 50  0000 C CNN
+F 2 "" H 4650 1550 50  0001 C CNN
+F 3 "" H 4650 1550 50  0001 C CNN
+	1    4650 1550
 	1    0    0    -1
 $EndComp
@@
 L Device:C C4
 U 1 1 5EF871B8
-P 4850 1900
-F 0 "C4" H 4900 2000 50  0000 L CNN
-F 1 "10uF" H 4900 1800 50  0000 L CNN
-F 2 "Capacitor_SMD:C_0805_2012Metric" H 4888 1750 50  0001 C CNN
-F 3 "~" H 4850 1900 50  0001 C CNN
-F 4 "C15850" H 4850 1900 50  0001 C CNN "LCSC"
-	1    4850 1900
+P 4650 1900
+F 0 "C4" H 4700 2000 50  0000 L CNN
+F 1 "10uF" H 4700 1800 50  0000 L CNN
+F 2 "Capacitor_SMD:C_0805_2012Metric" H 4688 1750 50  0001 C CNN
+F 3 "~" H 4650 1900 50  0001 C CNN
+F 4 "C15850" H 4650 1900 50  0001 C CNN "LCSC"
+	1    4650 1900
 	1    0    0    -1
 $EndComp
@@
 L Device:C C5
 U 1 1 5EF88469
-P 5950 1900
-F 0 "C5" H 6000 2000 50  0000 L CNN
-F 1 "10uF" H 6000 1800 50  0000 L CNN
-F 2 "Capacitor_SMD:C_0805_2012Metric" H 5988 1750 50  0001 C CNN
-F 3 "~" H 5950 1900 50  0001 C CNN
-F 4 "C15850" H 5950 1900 50  0001 C CNN "LCSC"
-	1    5950 1900
-	1    0    0    -1
-$EndComp
-Wire Wire Line
-	4850 2050 4850 2150
-Wire Wire Line
-	4850 2150 5400 2150
-Wire Wire Line
-	5950 2150 5950 2050
+P 6100 1900
+F 0 "C5" H 6150 2000 50  0000 L CNN
+F 1 "10uF" H 6150 1800 50  0000 L CNN
+F 2 "Capacitor_SMD:C_0805_2012Metric" H 6138 1750 50  0001 C CNN
+F 3 "~" H 6100 1900 50  0001 C CNN
+F 4 "C15850" H 6100 1900 50  0001 C CNN "LCSC"
+	1    6100 1900
+	1    0    0    -1
+$EndComp
+Wire Wire Line
+	4650 2050 4650 2150
+Wire Wire Line
+	4650 2150 5400 2150
+Wire Wire Line
+	6100 2150 6100 2050
 Wire Wire Line
 	5400 2250 5400 2150
 Connection ~ 5400 2150
 Wire Wire Line
-	5400 2150 5950 2150
+	5400 2150 6100 2150
 Wire Wire Line
 	5400 2150 5400 1950
 Wire Wire Line
-	4850 1550 4850 1650
-Wire Wire Line
-	5950 1550 5950 1650
-Wire Wire Line
-	5700 1650 5950 1650
-Connection ~ 5950 1650
-Wire Wire Line
-	5950 1650 5950 1750
-Wire Wire Line
-	5100 1650 4850 1650
-Connection ~ 4850 1650
-Wire Wire Line
-	4850 1650 4850 1750
+	4650 1550 4650 1650
+Wire Wire Line
+	6100 1550 6100 1650
+Wire Wire Line
+	5700 1650 6100 1650
+Connection ~ 6100 1650
+Wire Wire Line
+	6100 1650 6100 1750
+Wire Wire Line
+	5100 1650 4650 1650
+Connection ~ 4650 1650
+Wire Wire Line
+	4650 1650 4650 1750
 $Comp
 L Device:D_Schottky D1
@@
 	1    0    0    -1
 $EndComp
-Text GLabel 2950 2350 2    50   Input ~ 0
+Text GLabel 3800 2350 2    50   Input ~ 0
 D-
-Text GLabel 2950 2250 2    50   Input ~ 0
+Text GLabel 3800 2250 2    50   Input ~ 0
 D+
 $Comp
@@
 U 1 1 5EFEA4D2
 P 2400 4950
-F 0 "Y1" H 2250 5050 50  0000 C CNN
-F 1 "8MHz" H 2550 5050 50  0000 C CNN
+F 0 "Y1" H 2300 5100 50  0000 C CNN
+F 1 "8MHz" H 2500 5100 50  0000 C CNN
 F 2 "Crystal:Crystal_SMD_5032-2Pin_5.0x3.2mm" H 2400 4950 50  0001 C CNN
 F 3 "~" H 2400 4950 50  0001 C CNN
@@
 	2650 2250 1650 2250
 Wire Wire Line
-	1650 2350 2950 2350
-Wire Wire Line
-	2650 2250 2950 2250
+	1650 2350 3800 2350
+Wire Wire Line
+	2650 2250 3800 2250
 $Comp
 L Device:R R7
@@
 Wire Wire Line
 	5650 4550 5550 4550
+Text Notes 6350 3650 2    50   ~ 0
+Works with STM32F103C8,\nSTM32F103CB\nor GD32F103CB
 $EndSCHEMATC

Commit message: Cosmetic changes
Connections:
- no-connect marks 0 -> 17
Other:
- note added: "Works with STM32F103C8\nSTM32F103CB\nor GD32F103CB"
- note removed: "Works with STM32F103C8,\nSTM32F103CB\nor GD32F103CB"
Changed lines of the file:
@@
 Rev "b"
 Comp "Lars Boegild Thomsen"
-Comment1 "lbthomsen@gmail.com"
+Comment1 "lth@stm32world.com"
 Comment2 ""
 Comment3 ""
@@
 	5650 4550 5550 4550
 Text Notes 6350 3650 2    50   ~ 0
-Works with STM32F103C8,\nSTM32F103CB\nor GD32F103CB
+Works with STM32F103C8\nSTM32F103CB\nor GD32F103CB
+NoConn ~ 5200 5400
+NoConn ~ 3900 5400
+NoConn ~ 3900 5500
+NoConn ~ 3900 5600
+NoConn ~ 3900 5700
+NoConn ~ 3900 5800
+NoConn ~ 3900 5900
+NoConn ~ 3900 6000
+NoConn ~ 3900 6100
+NoConn ~ 3900 6200
+NoConn ~ 3900 6300
+NoConn ~ 3900 6400
+NoConn ~ 5200 5700
+NoConn ~ 5200 5800
+NoConn ~ 5200 5900
+NoConn ~ 5200 6000
+NoConn ~ 5200 6100
 $EndSCHEMATC
