File: pcb/stlink.kicad_sch (KiCad schematic)
At the start: 41 parts, among them J1 USB_A, Q1 S9013, U1 XC6206P332MR, U2 STM32F103C8, Y1 8MHz

Commit message: Hmmm
Parts:
- Y1: footprint Crystal:Crystal_SMD_5032-2Pin_5.0x3.2mm -> st-link:Crystal_SMD_5032-2Pin_5.0x3.2mm
Connections:
- no-connect marks 17 -> 19
Changed lines of the file:
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@@
   (no_connect (at 99.06 144.78))
   (no_connect (at 99.06 152.4))
+  (no_connect (at 99.06 172.72))
+  (no_connect (at 229.87 68.58))
   (no_connect (at 99.06 149.86))
   (wire (pts (xy 238.76 110.49) (xy 238.76 113.03))
@@
     (property "Reference" "Y1" (id 0) (at 58.42 121.92 0))
     (property "Value" "8MHz" (id 1) (at 63.5 121.92 0))
-    (property "Footprint" "Crystal:Crystal_SMD_5032-2Pin_5.0x3.2mm" (id 2) (at 60.96 125.73 0)
+    (property "Footprint" "st-link:Crystal_SMD_5032-2Pin_5.0x3.2mm" (id 2) (at 60.96 125.73 0)
       (effects (font (size 1.27 1.27)) hide)
     )
@@
     )
     (path "/00000000-0000-0000-0000-00005efea4d2"
-      (reference "Y1") (unit 1) (value "8MHz") (footprint "Crystal:Crystal_SMD_5032-2Pin_5.0x3.2mm")
-    )
-  )
+      (reference "Y1") (unit 1) (value "8MHz") (footprint "st-link:Crystal_SMD_5032-2Pin_5.0x3.2mm")
+    )
+  )

Commit message: Hmmmm
Parts:
- TP1, TP2, TP3, TP4, TP5: footprint TestPoint:TestPoint_Pad_D1.0mm -> TestPoint:TestPoint_Pad_1.0x1.0mm
Changed lines of the file:
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@@
       (effects (font (size 1.27 1.27)) (justify left))
     )
-    (property "Footprint" "TestPoint:TestPoint_Pad_D1.0mm" (id 2) (at 247.65 48.26 0)
+    (property "Footprint" "TestPoint:TestPoint_Pad_1.0x1.0mm" (id 2) (at 247.65 48.26 0)
       (effects (font (size 1.27 1.27)) hide)
     )
@@
       (effects (font (size 1.27 1.27)) (justify left))
     )
-    (property "Footprint" "TestPoint:TestPoint_Pad_D1.0mm" (id 2) (at 247.65 52.07 0)
+    (property "Footprint" "TestPoint:TestPoint_Pad_1.0x1.0mm" (id 2) (at 247.65 52.07 0)
       (effects (font (size 1.27 1.27)) hide)
     )
@@
       (effects (font (size 1.27 1.27)) (justify left))
     )
-    (property "Footprint" "TestPoint:TestPoint_Pad_D1.0mm" (id 2) (at 247.65 44.45 0)
+    (property "Footprint" "TestPoint:TestPoint_Pad_1.0x1.0mm" (id 2) (at 247.65 44.45 0)
       (effects (font (size 1.27 1.27)) hide)
     )
@@
       (effects (font (size 1.27 1.27)) (justify left))
     )
-    (property "Footprint" "TestPoint:TestPoint_Pad_D1.0mm" (id 2) (at 247.65 55.88 0)
+    (property "Footprint" "TestPoint:TestPoint_Pad_1.0x1.0mm" (id 2) (at 247.65 55.88 0)
       (effects (font (size 1.27 1.27)) hide)
     )
@@
       (effects (font (size 1.27 1.27)) (justify left))
     )
-    (property "Footprint" "TestPoint:TestPoint_Pad_D1.0mm" (id 2) (at 247.65 59.69 0)
+    (property "Footprint" "TestPoint:TestPoint_Pad_1.0x1.0mm" (id 2) (at 247.65 59.69 0)
       (effects (font (size 1.27 1.27)) hide)
     )
@@
     )
     (path "/00000000-0000-0000-0000-000060fae522"
-      (reference "TP1") (unit 1) (value "~") (footprint "TestPoint:TestPoint_Pad_D1.0mm")
+      (reference "TP1") (unit 1) (value "~") (footprint "TestPoint:TestPoint_Pad_1.0x1.0mm")
     )
     (path "/00000000-0000-0000-0000-00005efa2a39"
-      (reference "TP2") (unit 1) (value "~") (footprint "TestPoint:TestPoint_Pad_D1.0mm")
+      (reference "TP2") (unit 1) (value "~") (footprint "TestPoint:TestPoint_Pad_1.0x1.0mm")
     )
     (path "/00000000-0000-0000-0000-00005efad42c"
-      (reference "TP3") (unit 1) (value "~") (footprint "TestPoint:TestPoint_Pad_D1.0mm")
+      (reference "TP3") (unit 1) (value "~") (footprint "TestPoint:TestPoint_Pad_1.0x1.0mm")
     )
     (path "/00000000-0000-0000-0000-000060fae8e6"
-      (reference "TP4") (unit 1) (value "~") (footprint "TestPoint:TestPoint_Pad_D1.0mm")
+      (reference "TP4") (unit 1) (value "~") (footprint "TestPoint:TestPoint_Pad_1.0x1.0mm")
     )
     (path "/00000000-0000-0000-0000-000060faed81"
-      (reference "TP5") (unit 1) (value "~") (footprint "TestPoint:TestPoint_Pad_D1.0mm")
+      (reference "TP5") (unit 1) (value "~") (footprint "TestPoint:TestPoint_Pad_1.0x1.0mm")
     )
     (path "/00000000-0000-0000-0000-00005ef85b23"
