File: pcb/stlink.kicad_sch (KiCad schematic)
At the start: 41 parts, among them J1 USB_A, Q1 S9013, U1 XC6206P332MR, U2 STM32F103C8, Y1 8MHz

Commit message: Rev e order
Parts:
- U2: value STM32F103C8 -> STM32F103CB; LCSC C8734 -> C8304
Changed lines of the file:
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@@
     (in_bom yes) (on_board yes)
     (property "Reference" "U2" (id 0) (at 102.87 101.6 0))
-    (property "Value" "STM32F103C8" (id 1) (at 132.08 101.6 0))
+    (property "Value" "STM32F103CB" (id 1) (at 132.08 101.6 0))
     (property "Footprint" "Package_QFP:LQFP-48_7x7mm_P0.5mm" (id 2) (at 101.6 175.26 0)
       (effects (font (size 1.27 1.27)) (justify right) hide)
@@
       (effects (font (size 1.27 1.27)) hide)
     )
-    (property "LCSC" "C8734" (id 4) (at 116.84 139.7 0)
+    (property "LCSC" "C8304" (id 4) (at 116.84 139.7 0)
       (effects (font (size 1.27 1.27)) hide)
     )
@@
     )
     (path "/00000000-0000-0000-0000-00005ef826bc"
-      (reference "U2") (unit 1) (value "STM32F103C8") (footprint "Package_QFP:LQFP-48_7x7mm_P0.5mm")
+      (reference "U2") (unit 1) (value "STM32F103CB") (footprint "Package_QFP:LQFP-48_7x7mm_P0.5mm")
     )
     (path "/00000000-0000-0000-0000-00005efea4d2"

Commit message: Hmmmm
Connections:
- net T_CLK: now also U2.15 (PA5)
Changed lines of the file:
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@@
   (no_connect (at 99.06 160.02))
   (no_connect (at 132.08 137.16))
-  (no_connect (at 132.08 147.32))
   (no_connect (at 132.08 154.94))
   (no_connect (at 99.06 144.78))
@@
   (no_connect (at 99.06 172.72))
   (no_connect (at 229.87 68.58))
+  (no_connect (at 99.06 129.54))
   (no_connect (at 99.06 149.86))
   (wire (pts (xy 238.76 110.49) (xy 238.76 113.03))
@@
   )
   (wire (pts (xy 118.11 39.37) (xy 118.11 41.91))
+    (stroke (width 0) (type default) (color 0 0 0 0))
+  )
+  (wire (pts (xy 132.08 147.32) (xy 137.16 147.32))
     (stroke (width 0) (type default) (color 0 0 0 0))
   )
@@
       (effects (font (size 1.27 1.27)) hide)
     )
+  )
+  (global_label "T_CLK" (shape input) (at 137.16 147.32 0) (fields_autoplaced)
+    (effects (font (size 1.27 1.27)) (justify left))
+    (property "Intersheet References" "${INTERSHEET_REFS}" (id 0) (at 218.44 314.96 0)
+      (effects (font (size 1.27 1.27)) hide)
+    )
