File: pcb/stlink.kicad_sch (KiCad schematic)
At the start: 41 parts, among them J1 USB_A, Q1 S9013, U1 XC6206P332MR, U2 STM32F103CB, Y1 8MHz

Commit message: Hmmm
Parts:
- removed H1, H2, H3, H4: MouseBite, st-link:mouse-bite-1mm-slot, symbol st-link:MouseBite
Changed lines of the file:
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@@
     (pin "1")
-  )
-  (symbol (lib_id "st-link:MouseBite") (at 281.94 162.56 0) (unit 1)
-    (in_bom yes) (on_board yes)
-    (property "Reference" "H4" (id 0) (at 281.94 158.75 0)
-      (effects (font (size 1.27 1.27)) hide)
-    )
-    (property "Value" "MouseBite" (id 1) (at 281.94 166.37 0)
-      (effects (font (size 1.27 1.27)) hide)
-    )
-    (property "Footprint" "st-link:mouse-bite-1mm-slot" (id 2) (at 281.94 162.56 0)
-      (effects (font (size 1.27 1.27)) hide)
-    )
-    (property "Datasheet" "" (id 3) (at 281.94 162.56 0)
-      (effects (font (size 1.27 1.27)) hide)
-    )
-  )
-  (symbol (lib_id "st-link:MouseBite") (at 278.13 162.56 0) (unit 1)
-    (in_bom yes) (on_board yes)
-    (property "Reference" "H3" (id 0) (at 278.13 158.75 0)
-      (effects (font (size 1.27 1.27)) hide)
-    )
-    (property "Value" "MouseBite" (id 1) (at 278.13 166.37 0)
-      (effects (font (size 1.27 1.27)) hide)
-    )
-    (property "Footprint" "st-link:mouse-bite-1mm-slot" (id 2) (at 278.13 162.56 0)
-      (effects (font (size 1.27 1.27)) hide)
-    )
-    (property "Datasheet" "" (id 3) (at 278.13 162.56 0)
-      (effects (font (size 1.27 1.27)) hide)
-    )
-  )
-  (symbol (lib_id "st-link:MouseBite") (at 274.32 162.56 0) (unit 1)
-    (in_bom yes) (on_board yes)
-    (property "Reference" "H2" (id 0) (at 274.32 158.75 0)
-      (effects (font (size 1.27 1.27)) hide)
-    )
-    (property "Value" "MouseBite" (id 1) (at 274.32 166.37 0)
-      (effects (font (size 1.27 1.27)) hide)
-    )
-    (property "Footprint" "st-link:mouse-bite-1mm-slot" (id 2) (at 274.32 162.56 0)
-      (effects (font (size 1.27 1.27)) hide)
-    )
-    (property "Datasheet" "" (id 3) (at 274.32 162.56 0)
-      (effects (font (size 1.27 1.27)) hide)
-    )
-  )
-  (symbol (lib_id "st-link:MouseBite") (at 270.51 162.56 0) (unit 1)
-    (in_bom yes) (on_board yes)
-    (property "Reference" "H1" (id 0) (at 270.51 158.75 0)
-      (effects (font (size 1.27 1.27)) hide)
-    )
-    (property "Value" "MouseBite" (id 1) (at 270.51 166.37 0)
-      (effects (font (size 1.27 1.27)) hide)
-    )
-    (property "Footprint" "st-link:mouse-bite-1mm-slot" (id 2) (at 270.51 162.56 0)
-      (effects (font (size 1.27 1.27)) hide)
-    )
-    (property "Datasheet" "" (id 3) (at 270.51 162.56 0)
-      (effects (font (size 1.27 1.27)) hide)
-    )
   )
   (symbol (lib_id "Device:R") (at 90.17 165.1 270) (unit 1)
@@
       (reference "D3") (unit 1) (value "RED") (footprint "LED_SMD:LED_0603_1608Metric")
     )
-    (path "/00000000-0000-0000-0000-000060eb1e07"
-      (reference "H1") (unit 1) (value "MouseBite") (footprint "st-link:mouse-bite-1mm-slot")
-    )
-    (path "/00000000-0000-0000-0000-000060eb1b74"
-      (reference "H2") (unit 1) (value "MouseBite") (footprint "st-link:mouse-bite-1mm-slot")
-    )
-    (path "/00000000-0000-0000-0000-000060eb18bb"
-      (reference "H3") (unit 1) (value "MouseBite") (footprint "st-link:mouse-bite-1mm-slot")
-    )
-    (path "/00000000-0000-0000-0000-000060eb0ea1"
-      (reference "H4") (unit 1) (value "MouseBite") (footprint "st-link:mouse-bite-1mm-slot")
-    )
     (path "/00000000-0000-0000-0000-000060e6cec9"

Commit message: Hmmmm
Parts:
- J1: LCSC (none) -> C112454

Commit message: Hmmm
Other:
- note added: "Works with STM32F103C8 STM32F103CB or GD32F103CB But CB should be used"
- note removed: "Works with STM32F103C8 STM32F103CB or GD32F103CB"

Commit message: DFU Boot working
Changed lines of the file:
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@@
 (kicad_sch
-	(version 20231120)
+	(version 20250114)
 	(generator "eeschema")
-	(generator_version "8.0")
+	(generator_version "9.0")
 	(paper "A4")
 	(title_block
@@
 		(comment 3 "${AUTHOR_EMAIL}")
 	)
+	(text "Power Supply"
+		(exclude_from_sim no)
+		(at 113.03 15.24 0)
+		(effects
+			(font
+				(size 1.27 1.27)
+			)
+			(justify left bottom)
+		)
+	)
+	(text "Decoupling"
+		(exclude_from_sim no)
+		(at 168.91 15.24 0)
+		(effects
+			(font
+				(size 1.27 1.27)
+			)
+			(justify left bottom)
+		)
+	)
+	(text "USB Connection and renumeration circuitry"
+		(exclude_from_sim no)
+		(at 20.32 15.24 0)
+		(effects
+			(font
+				(size 1.27 1.27)
+			)
+			(justify left bottom)
+		)
+	)
+	(text "Programming Pins"
+		(exclude_from_sim no)
+		(at 218.44 15.24 0)
+		(effects
+			(font
+				(size 1.27 1.27)
+			)
+			(justify left bottom)
+		)
+	)
+	(text "Target Header"
+		(exclude_from_sim no)
+		(at 218.44 83.82 0)
+		(effects
+			(font
+				(size 1.27 1.27)
+			)
+			(justify left bottom)
+		)
+	)
+	(text "Works with STM32F103C8\nSTM32F103CB\nor GD32F103CB\nBut CB should be used"
+		(exclude_from_sim no)
+		(at 161.798 85.852 0)
+		(effects
+			(font
+				(size 1.27 1.27)
+			)
+			(justify right top)
+		)
+	)
+	(text "Two-color LED"
+		(exclude_from_sim no)
+		(at 168.91 83.82 0)
+		(effects
+			(font
+				(size 1.27 1.27)
+			)
+			(justify left bottom)
+		)
+	)
+	(text "MCU"
+		(exclude_from_sim no)
+		(at 20.32 83.82 0)
+		(effects
+			(font
+				(size 1.27 1.27)
+			)
+			(justify left bottom)
+		)
+	)
 	(junction
 		(at 194.31 38.1)
@@
 		)
 	)
-	(text "Power Supply"
-		(exclude_from_sim no)
-		(at 113.03 15.24 0)
-		(effects
-			(font
-				(size 1.27 1.27)
-			)
-			(justify left bottom)
-		)
-	)
-	(text "Decoupling"
-		(exclude_from_sim no)
-		(at 168.91 15.24 0)
-		(effects
-			(font
-				(size 1.27 1.27)
-			)
-			(justify left bottom)
-		)
-	)
-	(text "USB Connection and renumeration circuitry"
-		(exclude_from_sim no)
-		(at 20.32 15.24 0)
-		(effects
-			(font
-				(size 1.27 1.27)
-			)
-			(justify left bottom)
-		)
-	)
-	(text "Programming Pins"
-		(exclude_from_sim no)
-		(at 218.44 15.24 0)
-		(effects
-			(font
-				(size 1.27 1.27)
-			)
-			(justify left bottom)
-		)
-	)
-	(text "Target Header"
-		(exclude_from_sim no)
-		(at 218.44 83.82 0)
-		(effects
-			(font
-				(size 1.27 1.27)
-			)
-			(justify left bottom)
-		)
-	)
-	(text "Works with STM32F103C8\nSTM32F103CB\nor GD32F103CB\nBut CB should be used"
-		(exclude_from_sim no)
-		(at 161.798 85.852 0)
-		(effects
-			(font
-				(size 1.27 1.27)
-			)
-			(justify right top)
-		)
-	)
-	(text "Two-color LED"
-		(exclude_from_sim no)
-		(at 168.91 83.82 0)
-		(effects
-			(font
-				(size 1.27 1.27)
-			)
-			(justify left bottom)
-		)
-	)
-	(text "MCU"
-		(exclude_from_sim no)
-		(at 20.32 83.82 0)
-		(effects
-			(font
-				(size 1.27 1.27)
-			)
-			(justify left bottom)
-		)
-	)
 	(global_label "LED"
 		(shape input)
@@
 		)
 	)
+	(embedded_fonts no)
 )
