File: pcb2/stlink.kicad_sch (KiCad schematic)
At the start: 41 parts, among them J1 USB_C_Receptacle_USB2.0-Conne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, J2 IDC 2x5, Q1 S9013, U1 STM32F103CB, U3 AMS1117-3.3, Y1 8MHz

Commit message: Hmmmm
Parts:
- removed TP1, TP2, TP3, TP4, TP5: ~, TestPoint:TestPoint_Pad_1.0x1.0mm, symbol Connector:TestPoint
- added J3: Conn_01x05, Connector_PinHeader_2.54mm:PinHeader_1x05_P2.54mm_Vertical, symbol Connector_Generic:Conn_01x05
Connections:
- net +3V3: now also J3.1 (Pin_1)
- net B0: now also J3.4 (Pin_4)
- net CLK: now also J3.3 (Pin_3)
- net DIO: now also J3.2 (Pin_2)
- net GND: now also J3.5 (Pin_5)
Other:
- moved on the sheet: C10, C6, C7, C8, C9
