File: pcb2/stlink.kicad_sch (KiCad schematic)
At the start: 37 parts, among them J1 USB_A, Q1 S9013, U1 XC6206P332MR, U2 STM32F103CB, Y1 8MHz

Commit message: Hmmmm
Parts:
- removed J1: USB_A, st-link:USB_Male_A_UP2-AH-1-TH, symbol st-link:USB_A
- added J1: USB_C_Receptacle_USB2.0-Connector, st-link:USB_C_Receptacle_HRO_TYPE-C-31-M-12, symbol st-link:USB_C_Receptacle_USB2.0-Connector
- added R3, R4: 5k1, Resistor_SMD:R_0402_1005Metric, symbol Device:R
- renumbered R6 to R10, R9 to R11, R10 to R12, R11 to R13, R12 to R14, R13 to R15, R3 to R5, R7 to R6, R8 to R7, R4 to R8, R5 to R9, U2 to U1, U1 to U2
Connections:
- net D+: now also J1.A6 (D+), J1.B6 (D+)
- net D-: now also J1.A7 (D-), J1.B7 (D-)
- net GND: now also J1.A1 (GND), J1.A12 (GND), J1.B1 (GND), J1.B12 (GND), J1.S1 (SHIELD), R3.1, R4.1
- net VBUS: now also J1.A4 (VBUS), J1.A9 (VBUS), J1.B4 (VBUS), J1.B9 (VBUS)
- new net: J1.B5 (CC2), R3.2
- new net: J1.A5 (CC1), R4.2
- no-connect marks 19 -> 21
Other:
- moved on the sheet: D1, Q1, R10, R5, R8, R9

Commit message: Working on version 2
Parts:
- added H1, H2, H3, H4: MountingHole, MountingHole:MountingHole_2.2mm_M2, symbol Mechanical:MountingHole
- J2: footprint st-link:IDC_EDGE -> Connector_IDC:IDC-Header_2x05_P2.54mm_Vertical

Commit message: Hmmmmm
Parts:
- removed U2: XC6206P332MR, Package_TO_SOT_SMD:SOT-23, symbol Regulator_Linear:XC6206PxxxMR
- added C10: 100nF, Capacitor_SMD:C_0402_1005Metric, symbol Device:C
- added TP6: COVER, st-link:COVER, symbol Connector:TestPoint_Small
- added U3: AMS1117-3.3, Package_TO_SOT_SMD:SOT-223-3_TabPin2, symbol Regulator_Linear:AMS1117-3.3
- J2: value ~ -> IDC 2x5; footprint Connector_IDC:IDC-Header_2x05_P2.54mm_Vertical -> Connector_IDC:IDC-Header_2x05_P2.54mm_Vertical_SMD; LCSC (none) -> C41376028
- JP1: value ~ -> SolderJumper3
- TP1, TP2, TP3, TP4, TP5: now left out of the parts list
Connections:
- net +3V3: now also C10.1, U3.2 (VO)
- net +5V: now also U3.3 (VI)
- net GND: now also C10.2, U3.1 (GND)
Other:
- moved on the sheet: C6, C7, C8, C9

Commit message: Switching workstation
Parts:
- removed H1, H2, H3, H4: MountingHole, MountingHole:MountingHole_2.2mm_M2, symbol Mechanical:MountingHole
- removed TP6: COVER, st-link:COVER, symbol Connector:TestPoint_Small
- added B1: ~, st-link:BOARD, symbol st-link:Board
- U3: footprint Package_TO_SOT_SMD:SOT-223-3_TabPin2 -> st-link:SOT-223-3_TabPin2

Commit message: Order files ready for pcb2
Parts:
- J2: footprint Connector_IDC:IDC-Header_2x05_P2.54mm_Vertical_SMD -> st-link:IDC-Header_2x05_P2.54mm_Vertical_SMD
- Q1: footprint Package_TO_SOT_SMD:SOT-23 -> st-link:SOT-23
- U1: footprint Package_QFP:LQFP-48_7x7mm_P0.5mm -> st-link:LQFP-48_7x7mm_P0.5mm
Changed lines of the file:
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@@
 			)
 		)
-		(property "Footprint" "Package_QFP:LQFP-48_7x7mm_P0.5mm"
+		(property "Footprint" "st-link:LQFP-48_7x7mm_P0.5mm"
 			(at 101.6 175.26 0)
 			(effects
@@
 			)
 		)
-		(property "Footprint" "Connector_IDC:IDC-Header_2x05_P2.54mm_Vertical_SMD"
+		(property "Footprint" "st-link:IDC-Header_2x05_P2.54mm_Vertical_SMD"
 			(at 246.38 118.11 0)
 			(effects
@@
 			)
 		)
-		(property "Footprint" "Package_TO_SOT_SMD:SOT-23"
+		(property "Footprint" "st-link:SOT-23"
 			(at 68.58 33.02 0)
 			(effects
