File: pcb2/stlink.kicad_sch (KiCad schematic)
At the start: 37 parts, among them J1 USB_C_Receptacle_USB2.0-Conne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, J2 IDC 2x5, J3 Conn_01x05, Q1 S9013, U1 STM32F103CB, U3 AMS1117-3.3, Y1 8MHz

Commit message: Hmmmm
Parts:
- B1, R7: now not fitted; now left out of the parts list
- J3: now not fitted
- JP1: now left out of the parts list
Connections:
- net +3V3: now also J3.4 (Pin_4); no longer J3.1 (Pin_1)
- net B0: now also J3.5 (Pin_5); no longer J3.4 (Pin_4)
- net GND: now also J3.1 (Pin_1); no longer J3.5 (Pin_5)
Changed lines of the file:
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@@
 	(wire
 		(pts
-			(xy 254 41.91) (xy 256.54 41.91)
-		)
-		(stroke
-			(width 0)
-			(type default)
-		)
-	)
-	(wire
-		(pts
 			(xy 49.53 22.86) (xy 49.53 27.94)
 		)
@@
 	(wire
 		(pts
+			(xy 250.19 41.91) (xy 256.54 41.91)
+		)
+		(stroke
+			(width 0)
+			(type default)
+		)
+	)
+	(wire
+		(pts
 			(xy 44.45 127) (xy 44.45 123.19)
 		)
@@
 	(wire
 		(pts
-			(xy 254 39.37) (xy 254 41.91)
-		)
-		(stroke
-			(width 0)
-			(type default)
-		)
-	)
-	(wire
-		(pts
 			(xy 201.93 40.64) (xy 201.93 41.91)
 		)
@@
 		)
 	)
+	(wire
+		(pts
+			(xy 254 39.37) (xy 254 44.45)
+		)
+		(stroke
+			(width 0)
+			(type default)
+		)
+	)
 	(polyline
 		(pts
@@
 	(wire
 		(pts
-			(xy 256.54 46.99) (xy 252.73 46.99)
+			(xy 254 44.45) (xy 256.54 44.45)
 		)
 		(stroke
@@
 	(wire
 		(pts
-			(xy 115.57 180.34) (xy 115.57 182.88)
+			(xy 256.54 49.53) (xy 250.19 49.53)
 		)
 		(stroke
@@
 		)
 	)
-	(polyline
+	(wire
 		(pts
-			(xy 20.32 85.09) (xy 162.56 85.09)
+			(xy 115.57 180.34) (xy 115.57 182.88)
 		)
 		(stroke
@@
 		)
 	)
-	(wire
+	(polyline
 		(pts
-			(xy 256.54 49.53) (xy 252.73 49.53)
+			(xy 20.32 85.09) (xy 162.56 85.09)
 		)
 		(stroke
@@
 	(wire
 		(pts
-			(xy 252.73 44.45) (xy 256.54 44.45)
+			(xy 250.19 46.99) (xy 256.54 46.99)
 		)
 		(stroke
@@
 	(global_label "CLK"
 		(shape input)
-		(at 252.73 46.99 180)
+		(at 250.19 46.99 180)
 		(fields_autoplaced yes)
 		(effects
@@
 		)
 		(property "Intersheetrefs" "${INTERSHEET_REFS}"
-			(at 246.8309 46.99 0)
+			(at 244.2909 46.99 0)
 			(effects
 				(font
@@
 	(global_label "DIO"
 		(shape input)
-		(at 252.73 44.45 180)
+		(at 250.19 49.53 180)
 		(fields_autoplaced yes)
 		(effects
@@
 		)
 		(property "Intersheetrefs" "${INTERSHEET_REFS}"
-			(at 247.1937 44.45 0)
+			(at 244.6537 49.53 0)
 			(effects
 				(font
@@
 	(global_label "B0"
 		(shape input)
-		(at 252.73 49.53 180)
+		(at 250.19 41.91 180)
 		(fields_autoplaced yes)
 		(effects
@@
 		)
 		(property "Intersheetrefs" "${INTERSHEET_REFS}"
-			(at 247.9195 49.53 0)
+			(at 245.3795 41.91 0)
 			(effects
 				(font
@@
 		(unit 1)
 		(exclude_from_sim no)
-		(in_bom yes)
+		(in_bom no)
 		(on_board yes)
 		(dnp no)
@@
 		(unit 1)
 		(exclude_from_sim no)
-		(in_bom yes)
+		(in_bom no)
 		(on_board yes)
-		(dnp no)
+		(dnp yes)
 		(property "Reference" "R7"
 			(at 83.82 128.27 0)
@@
 		(unit 1)
 		(exclude_from_sim no)
-		(in_bom yes)
+		(in_bom no)
 		(on_board yes)
-		(dnp no)
+		(dnp yes)
 		(property "Reference" "B1"
 			(at 168.91 191.77 0)
@@
 		(lib_id "Connector_Generic:Conn_01x05")
 		(at 261.62 46.99 0)
+		(mirror x)
 		(unit 1)
 		(exclude_from_sim no)
 		(in_bom yes)
 		(on_board yes)
-		(dnp no)
-		(fields_autoplaced yes)
+		(dnp yes)
 		(property "Reference" "J3"
-			(at 264.16 45.7199 0)
+			(at 264.16 48.2601 0)
 			(effects
 				(font
@@
 		)
 		(property "Value" "Conn_01x05"
-			(at 264.16 48.2599 0)
+			(at 264.16 45.7201 0)
 			(effects
 				(font

Commit message: Hmmmm
Parts:
- Q1: symbol Device:Q_NPN_BEC -> Device:Q_NPN
Connections:
- net +3V3: now also Q1.C; no longer Q1.3 (C)
- net at R5.2: now also Q1.E; no longer Q1.2 (E)
- net at R10.2, R8.1, R9.2: now also Q1.B; no longer Q1.1 (B)
- no-connect marks 21 -> 20
Other:
- moved on the sheet: C1, C2, C3, JP1, R1, R11, R12, R13, R2, R6, R7, Y1

Commit message: Hmmmm
Connections:
- net GND: no longer J1.S1 (SHIELD)
- no-connect marks 20 -> 21
Other:
- note added: "Shield not connected!"
- note added: "T_PWR functionality depends on setting of JP1 Default T_PWR is ignored."
- note removed: "T_PWR functionality depends on setting of JP1"
Changed lines of the file:
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@@
 		)
 	)
-	(text "T_PWR functionality depends \non setting of JP1"
+	(text "T_PWR functionality depends \non setting of JP1\nDefault T_PWR is ignored."
 		(exclude_from_sim no)
-		(at 219.964 153.924 0)
+		(at 219.964 157.734 0)
 		(effects
 			(font
 				(size 1.27 1.27)
 			)
-			(justify left top)
+			(justify left bottom)
 		)
 	)
@@
 		)
 	)
+	(text "Shield not connected!"
+		(exclude_from_sim no)
+		(at 21.082 78.232 0)
+		(effects
+			(font
+				(size 1.27 1.27)
+			)
+			(justify left bottom)
+		)
+	)
 	(junction
 		(at 189.23 40.64)
@@
 	)
 	(no_connect
+		(at 24.13 66.04)
+	)
+	(no_connect
 		(at 87.63 146.05)
 	)
@@
 	(wire
 		(pts
-			(xy 100.33 58.42) (xy 66.04 58.42)
+			(xy 97.79 58.42) (xy 66.04 58.42)
 		)
 		(stroke
@@
 	(wire
 		(pts
-			(xy 71.12 55.88) (xy 100.33 55.88)
+			(xy 71.12 55.88) (xy 97.79 55.88)
 		)
 		(stroke
@@
 		)
 	)
-	(wire
-		(pts
-			(xy 24.13 66.04) (xy 24.13 68.58)
-		)
-		(stroke
-			(width 0)
-			(type default)
-		)
-	)
 	(polyline
 		(pts
@@
 	)
 	(global_label "LED"
-		(shape input)
+		(shape output)
 		(at 128.27 130.81 0)
 		(fields_autoplaced yes)
@@
 	)
 	(global_label "D-"
-		(shape input)
+		(shape bidirectional)
 		(at 128.27 135.89 0)
 		(fields_autoplaced yes)
@@
 		)
 		(property "Intersheetrefs" "${INTERSHEET_REFS}"
-			(at 133.4434 135.89 0)
+			(at 134.3959 135.89 0)
 			(effects
 				(font
@@
 	)
 	(global_label "T_RX"
-		(shape input)
+		(shape output)
 		(at 260.35 123.19 0)
 		(fields_autoplaced yes)
@@
 	)
 	(global_label "CLK"
-		(shape input)
+		(shape output)
 		(at 250.19 46.99 180)
 		(fields_autoplaced yes)
@@
 	)
 	(global_label "T_CLK"
-		(shape input)
+		(shape output)
 		(at 128.27 120.65 0)
 		(fields_autoplaced yes)
@@
 		)
 		(property "Intersheetrefs" "${INTERSHEET_REFS}"
-			(at 209.55 288.29 0)
+			(at 136.1043 120.65 0)
 			(effects
 				(font
 					(size 1.27 1.27)
 				)
+				(justify left)
 				(hide yes)
 			)
@@
 	)
 	(global_label "T_PWR"
-		(shape input)
+		(shape output)
 		(at 236.22 115.57 180)
 		(fields_autoplaced yes)
@@
 	)
 	(global_label "T_DIO"
-		(shape input)
+		(shape bidirectional)
 		(at 69.85 171.45 180)
 		(fields_autoplaced yes)
@@
 		)
 		(property "Intersheetrefs" "${INTERSHEET_REFS}"
-			(at 62.3785 171.45 0)
+			(at 61.426 171.45 0)
 			(effects
 				(font
@@
 	)
 	(global_label "T_SWO"
-		(shape input)
+		(shape bidirectional)
 		(at 236.22 120.65 180)
 		(fields_autoplaced yes)
@@
 		)
 		(property "Intersheetrefs" "${INTERSHEET_REFS}"
-			(at 227.9624 120.65 0)
+			(at 227.0099 120.65 0)
 			(effects
 				(font
@@
 	)
 	(global_label "T_RST"
-		(shape input)
+		(shape output)
 		(at 85.09 135.89 180)
 		(fields_autoplaced yes)
@@
 	)
 	(global_label "DIO"
-		(shape input)
+		(shape bidirectional)
 		(at 250.19 49.53 180)
 		(fields_autoplaced yes)
@@
 		)
 		(property "Intersheetrefs" "${INTERSHEET_REFS}"
-			(at 244.6537 49.53 0)
+			(at 243.7012 49.53 0)
 			(effects
 				(font
@@
 	)
 	(global_label "B0"
-		(shape input)
+		(shape output)
 		(at 250.19 41.91 180)
 		(fields_autoplaced yes)
@@
 	)
 	(global_label "D-"
-		(shape input)
-		(at 100.33 58.42 0)
+		(shape bidirectional)
+		(at 97.79 58.42 0)
 		(fields_autoplaced yes)
 		(effects
@@
 		)
 		(property "Intersheetrefs" "${INTERSHEET_REFS}"
-			(at 105.5034 58.42 0)
+			(at 103.9159 58.42 0)
 			(effects
 				(font
@@
 	)
 	(global_label "D+"
-		(shape input)
+		(shape bidirectional)
 		(at 128.27 138.43 0)
 		(fields_autoplaced yes)
@@
 		)
 		(property "Intersheetrefs" "${INTERSHEET_REFS}"
-			(at 133.4434 138.43 0)
+			(at 134.3959 138.43 0)
 			(effects
 				(font
@@
 	)
 	(global_label "T_DIO"
-		(shape input)
+		(shape bidirectional)
 		(at 260.35 118.11 0)
 		(fields_autoplaced yes)
@@
 		)
 		(property "Intersheetrefs" "${INTERSHEET_REFS}"
-			(at 267.8215 118.11 0)
+			(at 268.774 118.11 0)
 			(effects
 				(font
@@
 	)
 	(global_label "T_CLK"
-		(shape input)
+		(shape output)
 		(at 69.85 168.91 180)
 		(fields_autoplaced yes)
@@
 	)
 	(global_label "T_RX"
-		(shape input)
+		(shape output)
 		(at 128.27 115.57 0)
 		(fields_autoplaced yes)
@@
 	)
 	(global_label "D+"
-		(shape input)
-		(at 100.33 55.88 0)
+		(shape bidirectional)
+		(at 97.79 55.88 0)
 		(fields_autoplaced yes)
 		(effects
@@
 		)
 		(property "Intersheetrefs" "${INTERSHEET_REFS}"
-			(at 105.5034 55.88 0)
+			(at 103.9159 55.88 0)
 			(effects
 				(font
@@
 	)
 	(global_label "DIO"
-		(shape input)
+		(shape bidirectional)
 		(at 128.27 140.97 0)
 		(fields_autoplaced yes)
@@
 		)
 		(property "Intersheetrefs" "${INTERSHEET_REFS}"
-			(at 133.8063 140.97 0)
+			(at 134.7588 140.97 0)
 			(effects
 				(font
@@
 	)
 	(global_label "RENUM"
-		(shape input)
+		(shape output)
 		(at 128.27 146.05 0)
 		(fields_autoplaced yes)
@@
 	)
 	(global_label "T_SWO"
-		(shape input)
+		(shape bidirectional)
 		(at 128.27 133.35 0)
 		(fields_autoplaced yes)
@@
 		)
 		(property "Intersheetrefs" "${INTERSHEET_REFS}"
-			(at 136.5276 133.35 0)
+			(at 137.4801 133.35 0)
 			(effects
 				(font
@@
 					(unit 1)
 				)
-			)
-		)
-	)
-	(symbol
-		(lib_id "power:GND")
-		(at 24.13 68.58 0)
-		(unit 1)
-		(exclude_from_sim no)
-		(in_bom yes)
-		(on_board yes)
-		(dnp no)
-		(property "Reference" "#PWR01"
-			(at 24.13 74.93 0)
-			(effects
-				(font
-					(size 1.27 1.27)
-				)
-				(hide yes)
-			)
-		)
-		(property "Value" "GND"
-			(at 24.257 72.9742 0)
-			(effects
-				(font
-					(size 1.27 1.27)
-				)
-			)
-		)
-		(property "Footprint" ""
-			(at 24.13 68.58 0)
-			(effects
-				(font
-					(size 1.27 1.27)
-				)
-				(hide yes)
-			)
-		)
-		(property "Datasheet" ""
-			(at 24.13 68.58 0)
-			(effects
-				(font
-					(size 1.27 1.27)
-				)
-				(hide yes)
-			)
-		)
-		(property "Description" "Power symbol creates a global label with name \"GND\" , ground"
-			(at 24.13 68.58 0)
-			(effects
-				(font
-					(size 1.27 1.27)
-				)
-				(hide yes)
-			)
-		)
-		(pin "1"
-		)
-		(instances
-			(project "stlink"
-				(path "/240e5dac-6242-47a5-bbef-f76d11c715c0"
-					(reference "#PWR01")
-					(unit 1)
-				)

Commit message: Hmmm
Parts:
- R14, R15: value 220R -> 470R; LCSC C25091 -> C25117
Changed lines of the file:
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@@
 			)
 		)
-		(property "Value" "220R"
+		(property "Value" "470R"
 			(at 198.12 114.3 0)
 			(effects
@@
 			)
 		)
-		(property "LCSC" "C25091"
+		(property "LCSC" "C25117"
 			(at 191.77 113.03 90)
 			(effects
@@
 			)
 		)
-		(property "Value" "220R"
+		(property "Value" "470R"
 			(at 198.12 137.16 0)
 			(effects
@@
 			)
 		)
-		(property "LCSC" "C25091"
+		(property "LCSC" "C25117"
 			(at 191.77 135.89 90)
 			(effects
