File: pcb2/stlink.kicad_pcb (KiCad board)
At the start: 4 copper layers, 31 x 15 mm, 37 parts, among them J1 USB_A, Q1 S9013, U1 XC6206P332MR, U2 STM32F103CB, Y1 8MHz

Commit message: Hmmmm
Parts:
- added R3: 5k1, Resistor_SMD:R_0402_1005Metric, F.Cu at (164.9, 94.4)
- added R4: 5k1, Resistor_SMD:R_0402_1005Metric, F.Cu at (166.9, 94.4)
- J1: value USB_A -> USB_C_Receptacle_USB2.0-Connector; footprint st-link:USB_Male_A_UP2-AH-1-TH -> st-link:USB_C_Receptacle_HRO_TYPE-C-31-M-12
- moved D1 6.25 mm to (137.0, 83.8)
- moved J1 2.16 mm to (139.2, 90.0)
- renumbered R6 to R10, R9 to R11, R10 to R12, R11 to R13, R12 to R14, R13 to R15, R3 to R5, R7 to R6, R8 to R7, R4 to R8, R5 to R9, U2 to U1, U1 to U2
Routing:
- net VBUS: track 4.18 -> 0.00 mm
- net GND: vias 17 -> 13
Other:
- board size 31 x 15 mm -> 34.1 x 15 mm

Commit message: Working on version 2
Parts:
- added H1: MountingHole, MountingHole:MountingHole_2.2mm_M2, F.Cu at (104.1, 102.9)
- added H2: MountingHole, MountingHole:MountingHole_2.2mm_M2, F.Cu at (143.5, 102.9)
- added H3: MountingHole, MountingHole:MountingHole_2.2mm_M2, F.Cu at (143.5, 74.9)
- added H4: MountingHole, MountingHole:MountingHole_2.2mm_M2, F.Cu at (104.1, 74.9)
- J2: footprint st-link:IDC_EDGE -> Connector_IDC:IDC-Header_2x05_P2.54mm_Vertical; moved to F.Cu
- moved R4 55.6 mm to (111.8, 87.0), turned to -90 degrees
- moved R3 53.2 mm to (111.8, 91.4)
- moved C9 43.5 mm to (156.5, 110.3)
- moved R1 43.5 mm to (154.5, 110.3)
- moved J1 33.8 mm to (105.4, 88.9), turned to -90 degrees
- moved D1 28.6 mm to (113.7, 100.3)
- moved J2 28.0 mm to (136.5, 83.8), turned to 0 degrees
- moved U2 26.3 mm to (106.7, 80.0)
- moved TP2 23.6 mm to (116.8, 104.1)
- moved TP4 23.6 mm to (111.8, 104.1)
- moved TP1 22.5 mm to (121.9, 104.1)
- moved TP3 21.6 mm to (119.4, 104.1)
- moved TP5 21.6 mm to (114.3, 104.1)
- moved C5 20.3 mm to (111.1, 77.5)
- moved D2 19.5 mm to (132.7, 103.5), turned to -90 degrees
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Routing:
- net +5V: track 33.2 -> 0.00 mm, vias 2 -> 1
- net T_DIO: track 23.6 -> 0.00 mm, vias 2 -> 0
- net T_PWR: track 23.4 -> 0.00 mm
- net T_CLK: track 23.2 -> 0.00 mm, vias 2 -> 0
- net T_SWO: track 18.2 -> 0.00 mm
- net T_RST: track 15.7 -> 0.00 mm, vias 2 -> 1
- net T_RX: track 12.3 -> 0.00 mm, vias 2 -> 1
- net T_TX: track 9.58 -> 0.00 mm
- net Net-(U1-PC13): track 7.25 -> 0.00 mm
- net Net-(U1-PC14): track 6.60 -> 0.00 mm
- net LED: track 16.2 -> 11.2 mm
- net +3V3: track 28.0 -> 23.1 mm
- net Net-(U1-PB12): track 4.27 -> 0.00 mm
- net Net-(Q1-B): track 5.26 -> 1.75 mm
- net D-: track 7.72 -> 10.6 mm
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Other:
- board size 34.1 x 15 mm -> 44.5 x 33 mm
- board text added: "3.3V"

Commit message: Hmmmmm
Parts:
- removed U2: XC6206P332MR, Package_TO_SOT_SMD:SOT-23
- added C10: 100nF, Capacitor_SMD:C_0402_1005Metric, F.Cu at (121.9, 76.8)
- added TP6: COVER, st-link:COVER, F.Cu at (121.9, 69.2)
- added U3: AMS1117-3.3, Package_TO_SOT_SMD:SOT-223-3_TabPin2, F.Cu at (115.6, 77.5)
- J2: value ~ -> IDC 2x5; footprint Connector_IDC:IDC-Header_2x05_P2.54mm_Vertical -> Connector_IDC:IDC-Header_2x05_P2.54mm_Vertical_SMD
- JP1: value ~ -> SolderJumper3; moved to F.Cu
- TP1, TP2, TP3, TP4, TP5: moved to F.Cu
- moved C9 44.3 mm to (115.6, 93.3)
- moved R1 37.2 mm to (127.6, 84.5), turned to 0 degrees
- moved R14 28.4 mm to (116.2, 81.9), turned to 0 degrees
- moved D2 28.3 mm to (113.0, 83.2), turned to 180 degrees
- moved D3 25.6 mm to (113.0, 85.1), turned to 0 degrees
- moved R15 22.9 mm to (113.0, 87.0), turned to 90 degrees
- moved D1 19.3 mm to (108.0, 81.9), turned to 180 degrees
- moved C5 11.1 mm to (121.9, 74.9), turned to 0 degrees
- moved C4 7.01 mm to (108.6, 79.4)
- moved TP4 7.01 mm to (118.7, 103.5), turned to 180 degrees
- moved TP1 5.75 mm to (116.2, 103.5), turned to 180 degrees
- moved TP2 5.75 mm to (111.1, 103.5), turned to 180 degrees
- moved TP5 5.75 mm to (108.6, 103.5), turned to 180 degrees
- moved TP3 5.75 mm to (113.7, 103.5), turned to 180 degrees
- moved J2 5.24 mm to (137.8, 88.9)
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Routing:
- net +5V: track 0.00 -> 64.0 mm, vias 1 -> 2
- net T_DIO: track 0.00 -> 31.5 mm, vias 0 -> 2
- net T_RX: track 0.00 -> 28.0 mm, vias 1 -> 2
- net T_RST: track 0.00 -> 26.6 mm, vias 1 -> 2
- net T_TX: track 0.00 -> 24.9 mm, vias 1 -> 2
- net T_CLK: track 0.00 -> 21.8 mm, vias 0 -> 2
- net T_SWO: track 0.00 -> 18.5 mm, vias 1 -> 2
- net B0: track 2.18 -> 20.3 mm, vias 1 -> 0
- net CLK: track 0.00 -> 17.9 mm, vias 0 -> 2
- net VBUS: track 0.00 -> 15.9 mm
- net T_PWR: track 0.00 -> 12.9 mm
- net DIO: track 5.86 -> 18.0 mm, vias 1 -> 2
- net RENUM: track 10.8 -> 2.28 mm, vias 2 -> 0
- net +3V3: track 23.1 -> 29.7 mm, vias 10 -> 14
- net Net-(U1-PC13): track 0.00 -> 6.12 mm
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- added copper zone on F.Cu, net +3V3
Other:
- board text removed: "3.3V"
- board text removed: "5V/3V3"
- board text removed: "B0"
- board text removed: "CLK/DIO"
- board text removed: "GND"
- board text removed: "JLCJLCJLCJLC"
- board text removed: "PWR/GND"
- board text removed: "SWO/RST"
- board text removed: "TX/RX"

Commit message: Switching workstation
Parts:
- removed H1, H2, H3, H4: MountingHole, MountingHole:MountingHole_2.2mm_M2
- removed TP6: COVER, st-link:COVER
- added B1: ~, st-link:BOARD, F.Cu at (123.8, 88.9)
- U3: footprint Package_TO_SOT_SMD:SOT-223-3_TabPin2 -> st-link:SOT-223-3_TabPin2
- turned U3 to 180 degrees
Routing:
- net GND: vias 5 -> 8
- net +3V3: vias 14 -> 13

Commit message: Order files ready for pcb2
Parts:
- J2: footprint Connector_IDC:IDC-Header_2x05_P2.54mm_Vertical_SMD -> st-link:IDC-Header_2x05_P2.54mm_Vertical_SMD
- Q1: footprint Package_TO_SOT_SMD:SOT-23 -> st-link:SOT-23
- U1: footprint Package_QFP:LQFP-48_7x7mm_P0.5mm -> st-link:LQFP-48_7x7mm_P0.5mm
- moved R14 17.8 mm to (106.0, 96.5)
- moved D2 16.4 mm to (103.5, 96.5), turned to 0 degrees
- moved D3 16.4 mm to (103.5, 98.4), turned to 180 degrees
- moved R15 13.4 mm to (106.0, 98.4), turned to 180 degrees
- moved R11 3.70 mm to (114.3, 86.4), turned to -90 degrees
- moved Q1 2.69 mm to (110.5, 97.8), turned to 90 degrees
- moved R10 2.69 mm to (116.2, 97.2)
- moved R8 2.69 mm to (113.7, 99.1)
- moved R9 2.69 mm to (113.7, 97.2)
- moved J1 1.27 mm to (106.7, 88.9)
- turned J2 to -90 degrees
- turned U1 to 90 degrees
Routing:
- net LED: track 7.34 -> 30.8 mm, vias 0 -> 2
- net T_DIO: track 31.7 -> 28.1 mm
- net Net-(D2-A): track 3.98 -> 1.24 mm
- net Net-(U1-PB12): track 5.05 -> 2.31 mm
- net RENUM: track 2.28 -> 4.79 mm
- net Net-(Q1-E): track 4.10 -> 6.35 mm
- net +5V: track 64.0 -> 66.1 mm
- net CLK: track 17.9 -> 16.5 mm
- net Net-(U1-PA0): track 9.16 -> 10.6 mm
- net D+: track 12.4 -> 13.7 mm
- net T_RX: track 28.0 -> 29.2 mm
- net DIO: track 18.0 -> 19.2 mm
- net +3V3: track 29.7 -> 30.7 mm, vias 13 -> 15
- net GND: track 0.00 -> 0.76 mm, vias 8 -> 28

Commit message: Hmmmm
Parts:
- removed TP1, TP2, TP3, TP4, TP5: ~, TestPoint:TestPoint_Pad_1.0x1.0mm
- added J3: Conn_01x05, Connector_PinHeader_2.54mm:PinHeader_1x05_P2.54mm_Vertical, F.Cu at (108.6, 103.5)
Routing:
- net B0: track 20.3 -> 21.9 mm
- net +3V3: track 30.7 -> 29.4 mm, vias 15 -> 14
- net GND: vias 28 -> 27
Other:
- board text added: "B0"
- board text added: "GND"

Commit message: Tweaks
Parts:
- moved R2 11.4 mm to (116.2, 98.4), turned to 0 degrees
- moved R10 0.64 mm to (116.2, 96.5)
- moved R8 0.64 mm to (113.7, 98.4)
- moved R9 0.64 mm to (113.7, 96.5)
Routing:
- net B0: track 21.9 -> 14.3 mm
- net Net-(Q1-B): track 6.53 -> 7.93 mm
- net +5V: track 66.1 -> 65.5 mm
- net GND: vias 27 -> 36
