File: pcb2/stlink.kicad_pcb (KiCad board)
At the start: 4 copper layers, 44.5 x 33 mm, 37 parts, among them J1 USB_C_Receptacle_USB2.0-Conne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, J2 IDC 2x5, J3 Conn_01x05, Q1 S9013, U1 STM32F103CB, U3 AMS1117-3.3, Y1 8MHz

Commit message: Retried jobset export
Routing:
- net GND: vias 36 -> 37
Changed lines of the file:
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@@
 			(at 0 -2.38 90)
 			(layer "F.SilkS")
+			(hide yes)
 			(effects
 				(font
@@
 		(sheetname "/")
 		(sheetfile "stlink.kicad_sch")
-		(attr through_hole exclude_from_pos_files exclude_from_bom)
+		(attr through_hole exclude_from_pos_files)
 		(fp_line
 			(start -22.225 -13.97)
@@
 	)
 	(via
+		(at 114.3 90.932)
+		(size 0.6)
+		(drill 0.3)
+		(layers "F.Cu" "B.Cu")
+		(free yes)
+		(net 1)
+	)
+	(via
 		(at 114.3 74.93)
 		(size 0.6)
@@
 	)
 	(segment
-		(start 116.715 97.915)
-		(end 117.1575 97.4725)
+		(start 119.0625 97.4725)
+		(end 121.4 95.135)
 		(width 0.2286)
 		(layer "F.Cu")
@@
 	)
 	(segment
-		(start 116.715 98.425)
-		(end 116.715 99.57)
+		(start 116.715 97.915)
+		(end 117.1575 97.4725)
 		(width 0.2286)
 		(layer "F.Cu")
@@
 	)
 	(segment
-		(start 119.0625 97.4725)
-		(end 121.4 95.135)
+		(start 116.715 98.425)
+		(end 116.715 99.57)
 		(width 0.2286)
 		(layer "F.Cu")
@@
 	)
 	(segment
-		(start 116.715 99.57)
-		(end 118.745 101.6)
+		(start 116.715 98.425)
+		(end 116.715 97.915)
 		(width 0.2286)
 		(layer "F.Cu")
@@
 	)
 	(segment
-		(start 118.745 101.6)
-		(end 118.745 103.5)
+		(start 117.1575 97.4725)
+		(end 119.0625 97.4725)
 		(width 0.2286)
 		(layer "F.Cu")
@@
 	)
 	(segment
-		(start 117.1575 97.4725)
-		(end 119.0625 97.4725)
+		(start 121.4 95.135)
+		(end 121.4 93.0625)
 		(width 0.2286)
 		(layer "F.Cu")
@@
 	)
 	(segment
-		(start 116.715 98.425)
-		(end 116.715 97.915)
+		(start 116.715 99.57)
+		(end 118.745 101.6)
 		(width 0.2286)
 		(layer "F.Cu")
@@
 	)
 	(segment
-		(start 121.4 95.135)
-		(end 121.4 93.0625)
+		(start 118.745 101.6)
+		(end 118.745 103.5)
 		(width 0.2286)
 		(layer "F.Cu")
