File: pcb2/stlink.kicad_pcb (KiCad board)
At the start: 4 copper layers, 44.5 x 33 mm, 37 parts, among them J1 USB_C_Receptacle_USB2.0-Conne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, J2 IDC 2x5, J3 Conn_01x05, Q1 S9013, U1 STM32F103CB, U3 AMS1117-3.3, Y1 8MHz

Commit message: Hmmmm
Parts:
- moved C8 0.64 mm to (116.2, 83.8)
Connections:
- R10 pad 2: Net-(Q1-B) -> Net-(Q1-PadB)
- R5 pad 2: Net-(Q1-E) -> Net-(Q1-PadE)
- R8 pad 1: Net-(Q1-B) -> Net-(Q1-PadB)
- R9 pad 2: Net-(Q1-B) -> Net-(Q1-PadB)
Routing:
- net Net-(Q1-PadB): track 0.00 -> 7.93 mm
- net Net-(Q1-B): track 7.93 -> 0.00 mm
- net Net-(Q1-PadE): track 0.00 -> 7.39 mm
- net Net-(Q1-E): track 6.35 -> 0.00 mm
- net CLK: track 16.9 -> 12.2 mm
- net LED: track 30.8 -> 33.1 mm
- net DIO: track 19.5 -> 17.3 mm
- net GND: vias 37 -> 39

Commit message: Hmmmm
Parts:
- turned C2 to 180 degrees
- turned C3 to 180 degrees
Connections:
- J1 pad S1: GND -> unconnected-(J1-SHIELD-PadS1)_1
Routing:
- net +3V3: track 29.4 -> 32.5 mm
- net GND: vias 39 -> 41
- added copper zone on B.Cu, net +3V3
Other:
- board text added: "${TITLE}, rev. ${REVISION} ${YEAR} ${COMPANY}"

Commit message: Ready to order
Other:
- board text added: "${COMPANY}"
Changed lines of the file:
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@@
 	)
 	(gr_text "${TITLE}\nrev. ${REVISION}"
-		(at 140.97 104.14 0)
+		(at 141.605 104.14 0)
 		(layer "F.SilkS")
 		(effects
@@
 		)
 	)
+	(gr_text "${COMPANY}"
+		(at 141.605 73.025 0)
+		(layer "F.SilkS")
+		(effects
+			(font
+				(size 1 1)
+				(thickness 0.15)
+			)
+			(justify right top)
+		)
+	)
 	(gr_text "${TITLE}, rev. ${REVISION}\n${YEAR} ${COMPANY}"
-		(at 140.97 73.66 0)
+		(at 141.605 73.66 0)
 		(layer "B.SilkS")
 		(effects

Commit message: Ready for order
Routing:
- net GND: vias 41 -> 44
Changed lines of the file:
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@@
+	)
+	(via
+		(at 102.87 81.915)
+		(size 0.6)
+		(drill 0.3)
+		(layers "F.Cu" "B.Cu")
+		(free yes)
+		(net 1)
 	)
 	(via
@@
 	)
 	(via
+		(at 102.87 79.375)
+		(size 0.6)
+		(drill 0.3)
+		(layers "F.Cu" "B.Cu")
+		(free yes)
+		(net 1)
+	)
+	(via
 		(at 125.73 104.14)
 		(size 0.6)
@@
 		(size 0.6)
 		(drill 0.3)
+		(layers "F.Cu" "B.Cu")
+		(free yes)
+		(net 1)
+	)
+	(via
+		(at 120.65 82.55)
+		(size 0.6)
+		(drill 0.3)

Commit message: Jolt Connect rev. a files ready
Routing:
- net GND: vias 44 -> 43
Other:
- board text added: "${TITLE}, rev. ${REVISION}"
- board text added: "${TITLE}, rev. ${REVISION} ${DESC} ${YEAR} ${COMPANY}"
- board text removed: "${TITLE} rev. ${REVISION}"
- board text removed: "${TITLE}, rev. ${REVISION} ${YEAR} ${COMPANY}"
Changed lines of the file:
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@@
 	(property "AUTHOR_EMAIL" "lth@currentmakers.com")
 	(property "COMPANY" "CurrentMakers.com")
+	(property "DESC" "STM32 Programmer")
 	(property "REVISION" "a")
-	(property "TITLE" "STM32 Programmer 2")
+	(property "TITLE" "Jolt Connect")
 	(property "URL" "https://stm32world.com/wiki/DIY_STM32_Programmer_(ST-Link/V2-1)")
 	(property "YEAR" "2025")
@@
 		)
 	)
-	(gr_text "${TITLE}\nrev. ${REVISION}"
+	(gr_text "${TITLE}, rev. ${REVISION}"
 		(at 141.605 104.14 0)
 		(layer "F.SilkS")
@@
 		)
 	)
-	(gr_text "${TITLE}, rev. ${REVISION}\n${YEAR} ${COMPANY}"
-		(at 141.605 73.66 0)
+	(gr_text "${TITLE}, rev. ${REVISION}\n${DESC}\n${YEAR} ${COMPANY}"
+		(at 141.605 72.898 0)
 		(layer "B.SilkS")
 		(effects
@@
 		(size 0.6)
 		(drill 0.3)
-		(layers "F.Cu" "B.Cu")
-		(free yes)
-		(net 1)
-	)
-	(via
-		(at 127.635 104.14)
-		(size 0.6)
-		(drill 0.3)

Commit message: Hmmmm
Changed lines of the file:
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@@
 	(property "COMPANY" "CurrentMakers.com")
 	(property "DESC" "STM32 Programmer")
-	(property "REVISION" "a")
+	(property "REVISION" "b")
 	(property "TITLE" "Jolt Connect")
 	(property "URL" "https://stm32world.com/wiki/DIY_STM32_Programmer_(ST-Link/V2-1)")
@@
 		)
 		(pad "" np_thru_hole circle
-			(at -19.685 -13.97)
-			(size 2.2 2.2)
-			(drill 2.2)
+			(at -19.05 -13.335)
+			(size 3 3)
+			(drill 3)
 			(layers "F&B.Cu" "*.Mask")
 		)
 		(pad "" np_thru_hole circle
-			(at -19.685 13.97)
-			(size 2.2 2.2)
-			(drill 2.2)
+			(at -19.05 13.335)
+			(size 3 3)
+			(drill 3)
 			(layers "F&B.Cu" "*.Mask")
 		)
 		(pad "" np_thru_hole circle
-			(at 19.685 -13.97)
-			(size 2.2 2.2)
-			(drill 2.2)
+			(at 19.05 -13.335)
+			(size 3 3)
+			(drill 3)
 			(layers "F&B.Cu" "*.Mask")
 		)
 		(pad "" np_thru_hole circle
-			(at 19.685 13.97)
-			(size 2.2 2.2)
-			(drill 2.2)
+			(at 19.05 13.335)
+			(size 3 3)
+			(drill 3)
 			(layers "F&B.Cu" "*.Mask")
 		)
@@
 	)
 	(gr_text "${TITLE}, rev. ${REVISION}"
-		(at 141.605 104.14 0)
+		(at 140.335 104.775 0)
 		(layer "F.SilkS")
 		(effects
@@
 	)
 	(gr_text "${COMPANY}"
-		(at 141.605 73.025 0)
+		(at 140.335 73.025 0)
 		(layer "F.SilkS")
 		(effects
@@
 	)
 	(gr_text "${TITLE}, rev. ${REVISION}\n${DESC}\n${YEAR} ${COMPANY}"
-		(at 141.605 72.898 0)
+		(at 140.335 72.898 0)
 		(layer "B.SilkS")
 		(effects
@@
 	)
 	(via
-		(at 123.825 104.14)
+		(at 121.92 100.33)
 		(size 0.6)
 		(drill 0.3)
@@
 	)
 	(via
-		(at 106.045 100.965)
+		(at 107.315 100.965)
 		(size 0.6)
 		(drill 0.3)
@@
 	)
 	(via
-		(at 125.73 104.14)
+		(at 121.92 102.235)
 		(size 0.6)
 		(drill 0.3)

Commit message: Hmmmm
Routing:
- net T_RST: track 26.6 -> 31.0 mm
- net GND: vias 43 -> 44
Changed lines of the file:
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@@
 		)
 		(pad "" np_thru_hole circle
-			(at -19.05 -13.335)
+			(at -19.685 -13.97)
 			(size 3 3)
 			(drill 3)
@@
 		)
 		(pad "" np_thru_hole circle
-			(at -19.05 13.335)
+			(at -19.685 13.97)
 			(size 3 3)
 			(drill 3)
@@
 		)
 		(pad "" np_thru_hole circle
-			(at 19.05 -13.335)
+			(at 19.685 -13.97)
 			(size 3 3)
 			(drill 3)
@@
 		)
 		(pad "" np_thru_hole circle
-			(at 19.05 13.335)
+			(at 19.685 13.97)
 			(size 3 3)
 			(drill 3)
@@
 		)
 		(embedded_fonts no)
-		(model "${KIPRJMOD}/../cover/rev_a/cover.step"
+		(model "${KIPRJMOD}/../cover/rev_b/cover.step"
 			(opacity 0.5600)
 			(offset
-				(xyz -124 89 6)
+				(xyz -124 89 8)
 			)
 			(scale
@@
 	)
 	(via
+		(at 121.92 82.55)
+		(size 0.6)
+		(drill 0.3)
+		(layers "F.Cu" "B.Cu")
+		(free yes)
+		(net 1)
+	)
+	(via
 		(at 102.87 79.375)
 		(size 0.6)
@@
 	)
 	(via
-		(at 120.65 82.55)
+		(at 119.38 82.55)
 		(size 0.6)
 		(drill 0.3)
@@
 	)
 	(segment
-		(start 120.13715 86.65)
-		(end 116.4875 86.65)
+		(start 119.725 86.65)
+		(end 120.015 86.36)
 		(width 0.2286)
 		(layer "F.Cu")
@@
 	)
 	(segment
-		(start 120.88515 86.9277)
-		(end 120.41485 86.9277)
-		(width 0.2286)
-		(layer "F.Cu")
-		(net 9)
-	)
-	(segment
-		(start 120.41485 86.9277)
-		(end 120.13715 86.65)
-		(width 0.2286)
-		(layer "F.Cu")
-		(net 9)
-	)
-	(segment
-		(start 121.45285 86.36)
-		(end 120.88515 86.9277)
-		(width 0.2286)
-		(layer "F.Cu")
-		(net 9)
-	)
-	(segment
 		(start 121.92 86.36)
 		(end 122.4 85.88)
@@
 	)
 	(segment
-		(start 121.92 86.36)
-		(end 121.45285 86.36)
+		(start 120.015 86.36)
+		(end 121.92 86.36)
+		(width 0.2286)
+		(layer "F.Cu")
+		(net 9)
+	)
+	(segment
+		(start 116.4875 86.65)
+		(end 119.725 86.65)
 		(width 0.2286)
 		(layer "F.Cu")
@@
 	)
 	(segment
-		(start 120.9 86.11)
-		(end 120.65 86.36)
-		(width 0.2286)
-		(layer "F.Cu")
-		(net 13)
-	)
-	(segment
 		(start 120.9 84.7375)
-		(end 120.9 86.11)
+		(end 120.9 82.8)
 		(width 0.2286)
 		(layer "F.Cu")
@@
 		(net 13)
 	)
+	(segment
+		(start 120.9 82.8)
+		(end 120.65 82.55)
+		(width 0.2286)
+		(layer "F.Cu")
+		(net 13)
+	)
 	(via
 		(at 138.43 91.44)
@@
 	)
 	(via
-		(at 120.65 86.36)
+		(at 120.65 82.55)
 		(size 0.6)
 		(drill 0.3)
@@
 	)
 	(segment
-		(start 131.126793 90.488207)
-		(end 132.078586 91.44)
+		(start 120.65 89.535)
+		(end 120.65 82.55)
 		(width 0.2286)
 		(layer "B.Cu")
@@
 	)
 	(segment
-		(start 120.65 89.535)
-		(end 121.603207 90.488207)
+		(start 121.603207 90.488207)
+		(end 120.65 89.535)
 		(width 0.2286)
 		(layer "B.Cu")
@@
 	)
 	(segment
-		(start 120.65 86.36)
-		(end 120.65 89.535)
+		(start 131.126793 90.488207)
+		(end 121.603207 90.488207)
 		(width 0.2286)
 		(layer "B.Cu")
@@
 	)
 	(segment
-		(start 121.603207 90.488207)
-		(end 131.126793 90.488207)
+		(start 138.43 91.44)
+		(end 132.078586 91.44)
 		(width 0.2286)
 		(layer "B.Cu")
@@
 	(segment
 		(start 132.078586 91.44)
-		(end 138.43 91.44)
+		(end 131.126793 90.488207)
 		(width 0.2286)
 		(layer "B.Cu")

Commit message: Hmmm
Parts:
- R14, R15: value 220R -> 470R
Changed lines of the file:
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@@
 			)
 		)
-		(property "Value" "220R"
+		(property "Value" "470R"
 			(at 0 1.17 0)
 			(layer "F.Fab")
@@
 			)
 		)
-		(property "LCSC" "C25091"
+		(property "LCSC" "C25117"
 			(at 0 0 0)
 			(layer "F.Fab")
@@
 			)
 		)
-		(property "Value" "220R"
+		(property "Value" "470R"
 			(at 0 1.17 0)
 			(layer "F.Fab")
@@
 			)
 		)
-		(property "LCSC" "C25091"
+		(property "LCSC" "C25117"
 			(at 226.6 193.5 0)
 			(layer "F.Fab")
