File: pcb2/_autosave-stlink.kicad_pcb (KiCad board)
At the start: 4 copper layers, 44.5 x 33 mm, 37 parts, among them J1 USB_C_Receptacle_USB2.0-Conne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, J2 IDC 2x5, J3 Conn_01x05, Q1 S9013, U1 STM32F103CB, U3 AMS1117-3.3, Y1 8MHz

Commit message: Hmmmm
Parts:
- moved C8 0.64 mm to (116.2, 83.8)
Routing:
- net CLK: track 16.9 -> 12.6 mm
- net LED: track 30.8 -> 33.1 mm
- net DIO: track 19.5 -> 18.1 mm
- net Net-(Q1-E): track 6.35 -> 7.39 mm
Changed lines of the file:
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@@
 	(footprint "Capacitor_SMD:C_0402_1005Metric"
 		(layer "F.Cu")
-		(at 116.205 84.455 180)
+		(at 116.205 83.82 180)
 		(descr "Capacitor SMD 0402 (1005 Metric), square (rectangular) end terminal, IPC-7351 nominal, (Body size source: IPC-SM-782 page 76, https://www.pcb-3d.com/wordpress/wp-content/uploads/ipc-sm-782a_amendment_1_and_2.pdf), generated with kicad-footprint-generator")
 		(tags "capacitor")
@@
 	)
 	(via
+		(at 114.935 92.075)
+		(size 0.6)
+		(drill 0.3)
+		(layers "F.Cu" "B.Cu")
+		(free yes)
+		(net 1)
+	)
+	(via
 		(at 116.84 93.345)
 		(size 0.6)
@@
 	)
 	(via
-		(at 114.3 90.932)
-		(size 0.6)
-		(drill 0.3)
-		(layers "F.Cu" "B.Cu")
-		(free yes)
-		(net 1)
-	)
-	(via
 		(at 114.3 74.93)
 		(size 0.6)
@@
 	)
 	(segment
-		(start 116.685 84.935)
-		(end 116.84 85.09)
-		(width 0.2286)
-		(layer "F.Cu")
-		(net 3)
-	)
-	(segment
 		(start 116.078 92.456)
 		(end 116.078 93.317)
@@
 	)
 	(segment
+		(start 117.9 84.7375)
+		(end 117.1225 84.7375)
+		(width 0.2286)
+		(layer "F.Cu")
+		(net 3)
+	)
+	(segment
 		(start 141.595 83.82)
 		(end 141.595 82.56)
@@
 	)
 	(segment
-		(start 117.5475 85.09)
-		(end 117.9 84.7375)
+		(start 116.685 83.82)
+		(end 116.685 84.3)
 		(width 0.2286)
 		(layer "F.Cu")
@@
 	)
 	(segment
-		(start 116.84 85.09)
-		(end 117.5475 85.09)
+		(start 117.1225 84.7375)
+		(end 116.84 84.455)
 		(width 0.2286)
 		(layer "F.Cu")
@@
 	)
 	(segment
-		(start 116.685 84.455)
-		(end 116.685 84.935)
+		(start 116.685 84.3)
+		(end 116.84 84.455)
 		(width 0.2286)
 		(layer "F.Cu")
@@
 	)
 	(via
-		(at 116.84 85.09)
+		(at 116.84 84.455)
 		(size 0.6)
 		(drill 0.3)
@@
 	)
 	(segment
-		(start 114.3 99.06)
-		(end 113.284 100.076)
+		(start 113.665 94.615)
+		(end 114.3 95.25)
+		(width 0.2286)
+		(layer "B.Cu")
+		(net 7)
+	)
+	(segment
+		(start 113.665 90.17)
+		(end 113.665 94.615)
 		(width 0.2286)
 		(layer "B.Cu")
@@
 	(segment
 		(start 118.745 88.265)
-		(end 114.3 92.71)
+		(end 118.11 88.9)
 		(width 0.2286)
 		(layer "B.Cu")
@@
 	)
 	(segment
-		(start 114.3 92.71)
+		(start 114.3 99.06)
+		(end 113.284 100.076)
+		(width 0.2286)
+		(layer "B.Cu")
+		(net 7)
+	)
+	(segment
+		(start 114.3 95.25)
 		(end 114.3 99.06)
 		(width 0.2286)
@@
 	)
 	(segment
+		(start 114.935 88.9)
+		(end 113.665 90.17)
+		(width 0.2286)
+		(layer "B.Cu")
+		(net 7)
+	)
+	(segment
+		(start 118.11 88.9)
+		(end 114.935 88.9)
+		(width 0.2286)
+		(layer "B.Cu")
+		(net 7)
+	)
+	(segment
 		(start 120.578335 87.63)
 		(end 122.555 87.63)
@@
 	)
 	(segment
-		(start 117.9 91.65)
-		(end 117.9 93.0625)
+		(start 117.9 94.825)
+		(end 117.475 95.25)
 		(width 0.2286)
 		(layer "F.Cu")
@@
 	)
 	(segment
-		(start 118.11 91.44)
-		(end 117.9 91.65)
-		(width 0.2286)
-		(layer "F.Cu")
-		(net 10)
-	)
-	(segment
-		(start 118.745 91.44)
-		(end 118.11 91.44)
+		(start 117.9 93.0625)
+		(end 117.9 94.825)
 		(width 0.2286)
 		(layer "F.Cu")
@@
 	)
 	(via
-		(at 118.745 91.44)
+		(at 117.475 95.25)
 		(size 0.6)
 		(drill 0.3)
@@
 	(segment
 		(start 114.3 101.6)
-		(end 118.745 97.155)
+		(end 117.475 98.425)
 		(width 0.2286)
 		(layer "B.Cu")
@@
 	)
 	(segment
-		(start 113.665 101.6)
-		(end 114.3 101.6)
+		(start 117.475 95.25)
+		(end 117.475 98.425)
 		(width 0.2286)
 		(layer "B.Cu")
@@
 	)
 	(segment
-		(start 118.745 97.155)
-		(end 118.745 91.44)
+		(start 113.665 101.6)
+		(end 114.3 101.6)
 		(width 0.2286)
 		(layer "B.Cu")
@@
 	)
 	(segment
-		(start 125.095 85.09)
-		(end 125.095 85.8675)
+		(start 124.8125 86.15)
+		(end 124.8125 85.3725)
 		(width 0.2286)
 		(layer "F.Cu")
@@
 	)
 	(segment
-		(start 137.16 93.315)
-		(end 137.16 85.09)
+		(start 124.8125 85.3725)
+		(end 125.095 85.09)
 		(width 0.2286)
 		(layer "F.Cu")
@@
 	)
 	(segment
-		(start 133.995 93.98)
-		(end 136.495 93.98)
+		(start 137.16 93.315)
+		(end 137.16 85.09)
 		(width 0.2286)
 		(layer "F.Cu")
@@
 	)
 	(segment
-		(start 125.095 85.8675)
-		(end 124.8125 86.15)
+		(start 133.995 93.98)
+		(end 136.495 93.98)
 		(width 0.2286)
 		(layer "F.Cu")
@@
 	)
 	(segment
-		(start 117.63 90.65)
-		(end 118.11 90.17)
+		(start 114.455 90.65)
+		(end 114.3 90.805)
 		(width 0.2286)
 		(layer "F.Cu")
@@
 	(segment
 		(start 116.4875 90.65)
-		(end 117.63 90.65)
+		(end 114.455 90.65)
 		(width 0.2286)
 		(layer "F.Cu")
@@
 	)
 	(via
-		(at 118.11 90.17)
+		(at 114.3 90.805)
 		(size 0.6)
 		(drill 0.3)
@@
 	)
 	(segment
-		(start 118.11 97.155)
-		(end 116.84 98.425)
-		(width 0.2286)
-		(layer "B.Cu")
-		(net 16)
-	)
-	(segment
-		(start 115.57 98.425)
-		(end 116.84 98.425)
+		(start 111.125 101.6)
+		(end 112.395 101.6)
 		(width 0.2286)
 		(layer "B.Cu")
@@
 	)
 	(segment
-		(start 118.11 90.17)
-		(end 118.11 97.155)
+		(start 114.3 90.805)
+		(end 114.3 94.615)
 		(width 0.2286)
 		(layer "B.Cu")
@@
 	)
 	(segment
-		(start 111.76 101.6)
-		(end 112.395 101.6)
+		(start 114.3 94.615)
+		(end 115.57 95.885)
 		(width 0.2286)
 		(layer "B.Cu")
@@
 	)
 	(segment
-		(start 111.76 101.6)
-		(end 111.125 101.6)
+		(start 115.57 98.425)
+		(end 115.57 95.885)
 		(width 0.2286)
 		(layer "B.Cu")
@@
 	)
 	(segment
-		(start 113.03 92.202)
-		(end 113.03 91.95)
+		(start 112.649 94.361)
+		(end 110.871 94.361)
+		(width 0.2286)
+		(layer "F.Cu")
+		(net 25)
+	)
+	(segment
+		(start 113.03 93.98)
+		(end 112.649 94.361)
 		(width 0.2286)
 		(layer "F.Cu")
@@
 	)
 	(segment
+		(start 113.03 91.95)
+		(end 113.03 93.98)
+		(width 0.2286)
+		(layer "F.Cu")
+		(net 25)
+	)
+	(segment
 		(start 109.54 95.692)
-		(end 113.03 92.202)
+		(end 110.871 94.361)
 		(width 0.2286)
 		(layer "F.Cu")
