File: cover/cover.kicad_pcb (KiCad board)
At the start: 4 copper layers, 44.5 x 33 mm, 4 parts

Commit message: Syncing cover and pcb2
Routing:
- removed copper zone on In1.Cu, net (none)
- removed copper zone on In2.Cu, net (none)
Other:
- copper layers 4 -> 2
- board text added: "${YEAR} ${COMPANY}"
- board text added: "STM32 SWD"
- board text removed: "JLCJLCJLCJLC"
Changed lines of the file:
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@@
 	(layers
 		(0 "F.Cu" signal)
-		(4 "In1.Cu" signal)
-		(6 "In2.Cu" signal)
 		(2 "B.Cu" signal)
 		(9 "F.Adhes" user "F.Adhesive")
@@
 			)
 			(layer "dielectric 1"
-				(type "prepreg")
-				(thickness 0.1)
-				(material "FR4")
-				(epsilon_r 4.5)
-				(loss_tangent 0.02)
-			)
-			(layer "In1.Cu"
-				(type "copper")
-				(thickness 0.035)
-			)
-			(layer "dielectric 2"
 				(type "core")
-				(thickness 0.84)
-				(material "FR4")
-				(epsilon_r 4.5)
-				(loss_tangent 0.02)
-			)
-			(layer "In2.Cu"
-				(type "copper")
-				(thickness 0.035)
-			)
-			(layer "dielectric 3"
-				(type "prepreg")
-				(thickness 0.1)
+				(thickness 1.11)
 				(material "FR4")
 				(epsilon_r 4.5)
@@
 	(property "TITLE" "STM32 Programmer 2")
 	(property "URL" "https://stm32world.com/wiki/DIY_STM32_Programmer_(ST-Link/V2-1)")
+	(property "YEAR" "2025")
 	(net 0 "")
 	(footprint "MountingHole:MountingHole_2.2mm_M2"
@@
 	)
 	(gr_line
+		(start 129.54 100.33)
+		(end 142.24 100.33)
+		(stroke
+			(width 0.12)
+			(type default)
+		)
+		(layer "F.SilkS")
+	)
+	(gr_line
+		(start 129.54 77.47)
+		(end 142.24 77.47)
+		(stroke
+			(width 0.12)
+			(type default)
+		)
+		(layer "F.SilkS")
+	)
+	(gr_line
+		(start 129.54 77.47)
+		(end 129.54 100.33)
+		(stroke
+			(width 0.12)
+			(type default)
+		)
+		(layer "F.SilkS")
+	)
+	(gr_line
 		(start 123.825 110.49)
 		(end 123.825 63.5)
@@
 	)
 	(gr_text "${TITLE}\nrev. ${REVISION}"
-		(at 107.95 74.93 -0)
+		(at 107.95 73.66 0)
 		(layer "F.SilkS")
 		(effects
@@
 				(thickness 0.15)
 			)
-			(justify left)
+			(justify left top)
 		)
 	)
@@
 		)
 	)
+	(gr_text "STM32 SWD"
+		(at 129.032 88.9 90)
+		(layer "F.SilkS")
+		(effects
+			(font
+				(size 1 1)
+				(thickness 0.15)
+			)
+			(justify bottom)
+		)
+	)
+	(gr_text "${YEAR} ${COMPANY}"
+		(at 107.95 104.14 0)
+		(layer "F.SilkS")
+		(effects
+			(font
+				(size 1 1)
+				(thickness 0.15)
+			)
+			(justify left bottom)
+		)
+	)
 	(gr_text "GND"
 		(at 142.875 86.36 0)
@@
 			)
 			(justify right)
-		)
-	)
-	(gr_text "${TITLE}\nrev. ${REVISION}"
-		(at 140.335 74.93 0)
-		(layer "B.SilkS")
-		(effects
-			(font
-				(size 1 1)
-				(thickness 0.15)
-			)
-			(justify left mirror)
-		)
-	)
-	(gr_text "JLCJLCJLCJLC"
-		(at 140.335 104.14 0)
-		(layer "B.SilkS")
-		(effects
-			(font
-				(size 0.8 0.8)
-				(thickness 0.15)
-			)
-			(justify left mirror)
 		)
 	)
@@
 			(keep_text_aligned yes)
 		)
-		(gr_text "875.0000 mils"
+		(gr_text "22.2250 mm"
 			(at 134.9375 65.525 0)
 			(layer "Dwgs.User")
@@
 			(keep_text_aligned yes)
 		)
-		(gr_text "875.0000 mils"
+		(gr_text "22.2250 mm"
 			(at 112.7125 65.525 0)
 			(layer "Dwgs.User")
@@
 		(net 0)
 		(net_name "")
-		(layers "F.Cu" "B.Cu" "In2.Cu")
+		(layers "F.Cu" "B.Cu")
 		(hatch edge 0.508)
 		(connect_pads
@@
 			(thermal_gap 0.1524)
 			(thermal_bridge_width 0.3048)
+			(island_removal_mode 1)
+			(island_area_min 10)
 		)
 		(polygon
@@
 			)
 		)
-	)
-	(zone
-		(net 0)
-		(net_name "")
-		(layer "In1.Cu")
-		(hatch edge 0.508)
-		(connect_pads
-			(clearance 0.1524)
-		)
-		(min_thickness 0.1524)
-		(filled_areas_thickness no)
-		(fill yes
-			(thermal_gap 0.1524)
-			(thermal_bridge_width 0.3048)
-		)
-		(polygon
-			(pts
-				(xy 146.685 106.045) (xy 100.965 106.045) (xy 100.965 71.755) (xy 146.685 71.755)
-			)
-		)

Commit message: Tweaks
Other:
- board text added: "${TITLE}"
- board text added: "SWD"
- board text removed: "${TITLE} rev. ${REVISION}"
- board text removed: "STM32 SWD"
Changed lines of the file:
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@@
 	)
 	(gr_line
-		(start 129.54 100.33)
+		(start 129.794 100.33)
 		(end 142.24 100.33)
 		(stroke
@@
 	)
 	(gr_line
-		(start 129.54 77.47)
+		(start 142.24 77.47)
+		(end 145.796 77.47)
+		(stroke
+			(width 0.12)
+			(type default)
+		)
+		(layer "F.SilkS")
+	)
+	(gr_line
+		(start 129.794 77.47)
 		(end 142.24 77.47)
 		(stroke
@@
 	)
 	(gr_line
-		(start 129.54 77.47)
-		(end 129.54 100.33)
+		(start 145.796 100.33)
+		(end 142.24 100.33)
+		(stroke
+			(width 0.12)
+			(type default)
+		)
+		(layer "F.SilkS")
+	)
+	(gr_line
+		(start 129.794 77.47)
+		(end 129.794 100.33)
+		(stroke
+			(width 0.12)
+			(type default)
+		)
+		(layer "F.SilkS")
+	)
+	(gr_line
+		(start 145.796 77.47)
+		(end 145.796 100.33)
 		(stroke
 			(width 0.12)
@@
 		(layer "Edge.Cuts")
 	)
-	(gr_text "${TITLE}\nrev. ${REVISION}"
+	(gr_text "${TITLE}"
 		(at 107.95 73.66 0)
 		(layer "F.SilkS")
@@
 		)
 	)
-	(gr_text "STM32 SWD"
+	(gr_text "SWD"
 		(at 129.032 88.9 90)
 		(layer "F.SilkS")

Commit message: Hmmmm
Other:
- board text added: "JLCJLCJLCJLC"
Changed lines of the file:
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@@
 	(property "AUTHOR" "Lars Boegild Thomsen")
 	(property "AUTHOR_EMAIL" "lth@stm32world.com")
-	(property "COMPANY" "STM32World")
+	(property "COMPANY" "CurrentMakers.com")
 	(property "REVISION" "a")
 	(property "TITLE" "STM32 Programmer 2")
@@
 			)
 		)
-		(property "Datasheet" ""
+		(property "Datasheet" "~"
 			(at 0 0 0)
 			(layer "F.Fab")
@@
 			)
 		)
-		(property "Datasheet" ""
+		(property "Datasheet" "~"
 			(at 0 0 0)
 			(layer "F.Fab")
@@
 			)
 		)
-		(property "Datasheet" ""
+		(property "Datasheet" "~"
 			(at 0 0 0)
 			(layer "F.Fab")
@@
 			)
 		)
-		(property "Datasheet" ""
+		(property "Datasheet" "~"
 			(at 0 0 0)
 			(layer "F.Fab")
@@
 	)
 	(gr_line
-		(start 123.825 110.49)
-		(end 123.825 63.5)
+		(start 123.825 107.95)
+		(end 123.825 67.31)
 		(stroke
 			(width 0.1)
@@
 			)
 			(justify right)
+		)
+	)
+	(gr_text "JLCJLCJLCJLC"
+		(at 126.365 88.9 0)
+		(layer "B.SilkS")
+		(effects
+			(font
+				(size 0.8 0.8)
+				(thickness 0.15)
+				(bold yes)
+			)
+			(justify left mirror)
 		)
 	)
@@
 			(xy 101.6 72.39) (xy 101.6 105.41)
 		)
-		(height 12.5)
+		(height 3.81)
 		(format
 			(prefix "")
@@
 		)
 		(gr_text "33.0200 mm"
-			(at 87.95 88.9 90)
+			(at 96.64 88.9 90)
 			(layer "Dwgs.User")
 			(effects
@@
 			(xy 146.05 72.39) (xy 101.6 72.39)
 		)
-		(height 11.5)
+		(height 6.35)
 		(format
 			(prefix "")
@@
 		)
 		(gr_text "44.4500 mm"
-			(at 123.825 59.74 0)
+			(at 123.825 64.89 0)
 			(layer "Dwgs.User")
 			(effects
@@
 			(xy 123.825 72.39) (xy 146.05 72.39)
 		)
-		(height -5.715)
+		(height -3.175)
 		(orientation 0)
 		(format
@@
 		)
 		(gr_text "22.2250 mm"
-			(at 134.9375 65.525 0)
+			(at 134.9375 68.065 0)
 			(layer "Dwgs.User")
 			(effects
@@
 			(xy 101.6 72.39) (xy 123.825 72.39)
 		)
-		(height -5.715)
+		(height -3.175)
 		(orientation 0)
 		(format
@@
 		)
 		(gr_text "22.2250 mm"
-			(at 112.7125 65.525 0)
+			(at 112.7125 68.065 0)
 			(layer "Dwgs.User")
 			(effects
