File: cover/cover.kicad_pcb (KiCad board)
At the start: 2 copper layers, 44.5 x 33 mm, 4 parts

Commit message: Jolt Connect rev. a files ready
Other:
- board text added: "${TITLE} ${DESC}"
- board text removed: "${TITLE}"
Changed lines of the file:
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@@
 		(rev "${REVISION}")
 		(company "${COMPANY}")
-		(comment 1 "${URL}")
+		(comment 1 "${DESC}")
 		(comment 2 "${AUTHOR}")
 		(comment 3 "${AUTHOR_EMAIL}")
+		(comment 4 "${URL}")
 	)
 	(layers
@@
 	)
 	(property "AUTHOR" "Lars Boegild Thomsen")
-	(property "AUTHOR_EMAIL" "lth@stm32world.com")
+	(property "AUTHOR_EMAIL" "lth@currentmakers.com")
 	(property "COMPANY" "CurrentMakers.com")
+	(property "DESC" "STM32 Programmer")
 	(property "REVISION" "a")
-	(property "TITLE" "STM32 Programmer 2")
+	(property "TITLE" "Jolt Connect")
 	(property "URL" "https://stm32world.com/wiki/DIY_STM32_Programmer_(ST-Link/V2-1)")
 	(property "YEAR" "2025")
@@
 		(layer "Edge.Cuts")
 	)
-	(gr_text "${TITLE}"
+	(gr_text "${TITLE}\n${DESC}"
 		(at 107.95 73.66 0)
 		(layer "F.SilkS")

Commit message: Hmmmm
Parts:
- removed H1, H2, H3, H4: MountingHole, MountingHole:MountingHole_2.2mm_M2
- added B1: ~, st-link:BOARD, F.Cu at (123.8, 88.9)
Other:
- outline, holes or cut-outs redrawn

Commit message: Hmmmm
Changed lines of the file:
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@@
 		(sheetname "/")
 		(sheetfile "cover.kicad_sch")
-		(attr through_hole dnp)
+		(attr through_hole exclude_from_bom dnp)
 		(fp_line
 			(start -22.225 -13.97)
@@
 		)
 		(pad "" np_thru_hole circle
-			(at -19.05 -13.335)
+			(at -19.685 -13.97)
 			(size 3 3)
 			(drill 3)
@@
 		)
 		(pad "" np_thru_hole circle
-			(at -19.05 13.335)
+			(at -19.685 13.97)
 			(size 3 3)
 			(drill 3)
@@
 		)
 		(pad "" np_thru_hole circle
-			(at 19.05 -13.335)
+			(at 19.685 -13.97)
 			(size 3 3)
 			(drill 3)
@@
 		)
 		(pad "" np_thru_hole circle
-			(at 19.05 13.335)
+			(at 19.685 13.97)
 			(size 3 3)
 			(drill 3)
@@
 	)
 	(gr_line
-		(start 129.794 100.33)
-		(end 142.24 100.33)
+		(start 129.794 99.695)
+		(end 142.24 99.695)
 		(stroke
 			(width 0.12)
@@
 	)
 	(gr_line
-		(start 142.24 77.47)
-		(end 145.796 77.47)
+		(start 142.24 78.105)
+		(end 145.796 78.105)
 		(stroke
 			(width 0.12)
@@
 	)
 	(gr_line
-		(start 129.794 77.47)
-		(end 142.24 77.47)
+		(start 129.794 78.105)
+		(end 142.24 78.105)
 		(stroke
 			(width 0.12)
@@
 	)
 	(gr_line
-		(start 145.796 100.33)
-		(end 142.24 100.33)
+		(start 145.796 99.695)
+		(end 142.24 99.695)
 		(stroke
 			(width 0.12)
@@
 	)
 	(gr_line
-		(start 129.794 77.47)
-		(end 129.794 100.33)
+		(start 129.794 78.105)
+		(end 129.794 99.695)
 		(stroke
 			(width 0.12)
@@
 	)
 	(gr_line
-		(start 145.796 77.47)
-		(end 145.796 100.33)
+		(start 145.796 78.105)
+		(end 145.796 99.695)
 		(stroke
 			(width 0.12)
